Commit message: Added Blender-based wheels and an SDF version of the model for use in Gazebo

File: packages/ai_swarm/ez_rassor_description/urdf_depricated/ez_rassor.xacro (robot description, xacro)
@@ -27,5 +27,5 @@
       <origin xyz="0 0 0" rpy="0 1.5707 1.5707"/>
       <geometry>
-        <cylinder radius="0.1" length="0.05"/>
+          <mesh filename="package://ez_rassor_description/meshes/wheel.dae"/>
       </geometry>
     </collision>
@@ -33,5 +33,5 @@
       <origin xyz="0 0 0" rpy="0 1.5707 1.5707"/>
       <geometry>
-        <cylinder radius="0.1" length="0.05"/>
+          <mesh filename="package://ez_rassor_description/meshes/wheel.dae"/>
       </geometry>
     </visual>
@@ -46,5 +46,5 @@
       <origin xyz="0 0 0" rpy="0 1.5707 1.5707"/>
       <geometry>
-        <cylinder radius="0.1" length="0.05"/>
+          <mesh filename="package://ez_rassor_description/meshes/wheel.dae"/>
       </geometry>
     </collision>
@@ -52,5 +52,5 @@
       <origin xyz="0 0 0" rpy="0 1.5707 1.5707"/>
       <geometry>
-        <cylinder radius="0.1" length="0.05"/>
+          <mesh filename="package://ez_rassor_description/meshes/wheel.dae"/>
       </geometry>
     </visual>
@@ -65,5 +65,5 @@
       <origin xyz="0 0 0" rpy="0 1.5707 1.5707"/>
       <geometry>
-        <cylinder radius="0.1" length="0.05"/>
+          <mesh filename="package://ez_rassor_description/meshes/wheel.dae"/>
       </geometry>
     </collision>
@@ -71,5 +71,5 @@
       <origin xyz="0 0 0" rpy="0 1.5707 1.5707"/>
       <geometry>
-        <cylinder radius="0.1" length="0.05"/>
+          <mesh filename="package://ez_rassor_description/meshes/wheel.dae"/>
       </geometry>
     </visual>
@@ -84,5 +84,5 @@
       <origin xyz="0 0 0" rpy="0 1.5707 1.5707"/>
       <geometry>
-        <cylinder radius="0.1" length="0.05"/>
+          <mesh filename="package://ez_rassor_description/meshes/wheel.dae"/>
       </geometry>
     </collision>
@@ -90,5 +90,5 @@
       <origin xyz="0 0 0" rpy="0 1.5707 1.5707"/>
       <geometry>
-        <cylinder radius="0.1" length="0.05"/>
+          <mesh filename="package://ez_rassor_description/meshes/wheel.dae"/>
       </geometry>
     </visual>
