Commit message: Added stereo cameras to front and back of robot
Cameras are mounted to 'base_link' so they will stay in position when the arms move. Robot currently has inertial problems that need to be resolved before it can move.

File: packages/ai_swarm/depreciated/ez_rassor_description/urdf/ez_rassor.xacro (robot description, xacro)
@@ -1,20 +1,13 @@
 <?xml version='1.0'?>
 <robot name="ez_rassor" xmlns:xacro="http://www.ros.org/wiki/xacro">
-  <xacro:property name="cameraSize" value="0.05"/>
-  <xacro:property name="cameraMass" value="0.1"/>
-  <xacro:include filename="$(find ez_rassor_description)/urdf/ez_rassor.gazebo" />
-  <xacro:include filename="$(find ez_rassor_description)/urdf/materials.xacro" />
-  <xacro:include filename="$(find ez_rassor_description)/urdf/macros.xacro" />
-  <!--Below are all of the robot's Links/-->
+ <xacro:include filename="$(find ez_rassor_description)/urdf/ez_rassor.gazebo" />
+ <xacro:include filename="$(find ez_rassor_description)/urdf/materials.xacro" />
+ <xacro:include filename="$(find ez_rassor_description)/urdf/macros.xacro" />
   <link name='base_link'>
     <pose>0 0 0.1 0 0 0</pose>
     <inertial>
-      <mass value="10.0"/>
+      <mass value="1.0"/>
       <origin xyz="0.0 0 0.1" rpy=" 0 0 0"/>
-      <inertia
-          ixx="0.5" ixy="0" ixz="0"
-          iyy="1.0" iyz="0"
-          izz="0.1"
-      />
+      <box_inertia m="1.0" x=".4" y=".2" z=".1"/>
     </inertial>
     <collision name='collision'>
@@ -45,10 +38,6 @@
     <inertial>
       <origin xyz="0 0 0" rpy="0 1.5707 1.5707"/>
-      <mass value="5"/>
-      <cylinder_inertia m="5" r="0.1" h="0.05"/>
-      <inertia
-        ixx="1.0" ixy="0.0" ixz="0.0"
-        iyy="1.0" iyz="0.0"
-        izz="1.0"/>
+      <mass value=".5"/>
+      <cylinder_inertia m=".5" r="0.1" h="0.05"/>
     </inertial>
   </link>
@@ -68,10 +57,6 @@
     <inertial>
       <origin xyz="0 0 0" rpy="0 1.5707 1.5707"/>
-      <mass value="5"/>
-      <cylinder_inertia m="5" r="0.1" h="0.05"/>
-      <inertia
-        ixx="1.0" ixy="0.0" ixz="0.0"
-        iyy="1.0" iyz="0.0"
-        izz="1.0"/>
+      <mass value=".5"/>
+      <cylinder_inertia m=".5" r="0.1" h="0.05"/>
     </inertial>
   </link>
@@ -91,10 +76,6 @@
     <inertial>
       <origin xyz="0 0 0" rpy="0 1.5707 1.5707"/>
-      <mass value="5"/>
-      <cylinder_inertia m="5" r="0.1" h="0.05"/>
-      <inertia
-        ixx="1.0" ixy="0.0" ixz="0.0"
-        iyy="1.0" iyz="0.0"
-        izz="1.0"/>
+      <mass value=".5"/>
+      <cylinder_inertia m=".5" r="0.1" h="0.05"/>
     </inertial>
   </link>
@@ -114,10 +95,6 @@
     <inertial>
       <origin xyz="0 0 0" rpy="0 1.5707 1.5707"/>
-      <mass value="5"/>
-      <cylinder_inertia m="5" r="0.1" h="0.05"/>
-      <inertia
-        ixx="1.0" ixy="0.0" ixz="0.0"
-        iyy="1.0" iyz="0.0"
-        izz="1.0"/>
+      <mass value=".5"/>
+      <cylinder_inertia m=".5" r="0.1" h="0.05"/>
     </inertial>
   </link>
@@ -137,10 +114,6 @@
     <inertial>
       <origin xyz="0 0 0" rpy="0 1.5707 1.5707"/>
-      <mass value="5"/>
-      <cylinder_inertia m="5" r="0.1" h="0.05"/>
-      <inertia
-        ixx="1.0" ixy="0.0" ixz="0.0"
-        iyy="1.0" iyz="0.0"
-        izz="1.0"/>
+      <mass value=".5"/>
+      <cylinder_inertia m=".5" r="0.1" h="0.05"/>
     </inertial>
   </link>
@@ -160,10 +133,6 @@
     <inertial>
       <origin xyz="0 0 0" rpy="0 1.5707 1.5707"/>
-      <mass value="5"/>
-      <cylinder_inertia m="5" r="0.1" h="0.05"/>
-      <inertia
-        ixx="1.0" ixy="0.0" ixz="0.0"
-        iyy="1.0" iyz="0.0"
-        izz="1.0"/>
+      <mass value=".5"/>
+      <cylinder_inertia m=".5" r="0.1" h="0.05"/>
     </inertial>
   </link>
@@ -172,5 +141,5 @@
       <origin xyz="0 0 0" rpy="0 1.5707 1.5707"/>
       <geometry>
-        <cylinder radius="0.1" length="0.05"/>
+        <cylinder radius="0.07" length="0.05"/>
       </geometry>
     </collision>
@@ -183,10 +152,6 @@
     <inertial>
       <origin xyz="0 0 0" rpy="0 1.5707 1.5707"/>
-      <mass value="5"/>
-      <cylinder_inertia m="5" r="0.1" h="0.05"/>
-      <inertia
-        ixx="1.0" ixy="0.0" ixz="0.0"
-        iyy="1.0" iyz="0.0"
-        izz="1.0"/>
+      <mass value="10"/>
+      <cylinder_inertia m="10" r="0.1" h="0.05"/>
     </inertial>
   </link>
@@ -195,5 +160,5 @@
       <origin xyz="0 0 0" rpy="0 1.5707 1.5707"/>
       <geometry>
-        <cylinder radius="0.1" length="0.05"/>
+        <cylinder radius="0.07" length="0.05"/>
       </geometry>
     </collision>
@@ -206,18 +171,13 @@
     <inertial>
       <origin xyz="0 0 0" rpy="0 1.5707 1.5707"/>
-      <mass value="5"/>
-      <cylinder_inertia m="5" r="0.1" h="0.05"/>
-      <inertia
-        ixx="1.0" ixy="0.0" ixz="0.0"
-        iyy="1.0" iyz="0.0"
-        izz="1.0"/>
-    </inertial>
-  </link>
-  <!--First Camera Added/-->
-  <link name="f_stereo_1">
+      <mass value="10"/>
+      <cylinder_inertia m="10" r="0.1" h="0.05"/>
+    </inertial>
+  </link>
+  <link name="camera_back">
     <collision>
-      <origin xyz="0 0 0" rpy="0 0 0"/>
-      <geometry>
-        <box size="${cameraSize} ${cameraSize} ${cameraSize}"/>
+      <origin xyz="0 0 0" rpy="0 1.57 1.57"/>
+      <geometry>
+    <box size=".1 .1 .1"/>
       </geometry>
     </collision>
@@ -225,105 +185,59 @@
       <origin xyz="0 0 0" rpy="0 0 0"/>
       <geometry>
-        <box size="${cameraSize} ${cameraSize} ${cameraSize}"/>
-      </geometry>
-      <material name="green"/>
-    </visual>
-    <inertial>
-      <mass value="${cameraMass}" />
+    <box size=".1 .1 .1"/>
+      </geometry>
+      <material name="red"/>
+    </visual>
+    <inertial>
+      <mass value="1e-5" />
       <origin xyz="0 0 0" rpy="0 0 0"/>
-      <box_inertia m="${cameraMass}" x="${cameraSize}" y="${cameraSize}" z="${cameraSize}" />
-      <inertia ixx="1e-6" ixy="0" ixz="0" iyy="1e-6" iyz="0" izz="1e-6" />
-    </inertial>
-  </link>
-  <!--Second Camera Added/-->
-  <link name="f_stereo_2">
-    <collision>
-      <origin xyz="0 0 0" rpy="0 0 0"/>
-      <geometry>
-        <box size="${cameraSize} ${cameraSize} ${cameraSize}"/>
-      </geometry>
-    </collision>
-    <visual>
-      <origin xyz="0 0 0" rpy="0 0 0"/>
-      <geometry>
-        <box size="${cameraSize} ${cameraSize} ${cameraSize}"/>
-      </geometry>
-      <material name="green"/>
-    </visual>
-    <inertial>
-      <mass value="${cameraMass}" />
-      <origin xyz="0 0 0" rpy="0 0 0"/>
-      <box_inertia m="${cameraMass}" x="${cameraSize}" y="${cameraSize}" z="${cameraSize}" />
-      <inertia ixx="1e-6" ixy="0" ixz="0" iyy="1e-6" iyz="0" izz="1e-6" />
-    </inertial>
-  </link>
-    <!--Third Camera Added/-->
-  <link name="f_stereo_3">
-    <collision>
-      <origin xyz="0 0 0" rpy="0 0 0"/>
-      <geometry>
-        <box size="${cameraSize} ${cameraSize} ${cameraSize}"/>
-      </geometry>
-    </collision>
-    <visual>
-      <origin xyz="0 0 0" rpy="0 0 0"/>
-      <geometry>
-        <box size="${cameraSize} ${cameraSize} ${cameraSize}"/>
-      </geometry>
-      <material name="green"/>
-    </visual>
-    <inertial>
-      <mass value="${cameraMass}" />
-      <origin xyz="0 0 0" rpy="0 0 0"/>
-      <box_inertia m="${cameraMass}" x="${cameraSize}" y="${cameraSize}" z="${cameraSize}" />
-      <inertia ixx="1e-6" ixy="0" ixz="0" iyy="1e-6" iyz="0" izz="1e-6" />
-    </inertial>
-  </link>
-      <!--Fourth Camera Added/-->
-  <link name="f_stereo_4">
-    <collision>
-      <origin xyz="0 0 0" rpy="0 0 0"/>
-      <geometry>
-        <box size="${cameraSize} ${cameraSize} ${cameraSize}"/>
-      </geometry>
-    </collision>
-    <visual>
-      <origin xyz="0 0 0" rpy="0 0 0"/>
-      <geometry>
-        <box size="${cameraSize} ${cameraSize} ${cameraSize}"/>
-      </geometry>
-      <material name="green"/>
-    </visual>
-    <inertial>
-      <mass value="${cameraMass}" />
-      <origin xyz="0 0 0" rpy="0 0 0"/>
-      <box_inertia m="${cameraMass}" x="${cameraSize}" y="${cameraSize}" z="${cameraSize}" />
-      <inertia ixx="1e-6" ixy="0" ixz="0" iyy="1e-6" iyz="0" izz="1e-6" />
-    </inertial>
-  </link>
-  <!--Below are all of the robot's joints/-->
+      <box_inertia m="1e-5" x=".1" y = ".1" z=".1"/>
+    </inertial>
+  </link>
+  <transmission name="left_wheel_back_tran">
+    <type>transmission_interface/SimpleTransmission</type>
+    <joint name="left_wheel_back_hinge">
+      <hardwareInterface>hardware_interface/EffortJointInterface</hardwareInterface>
+    </joint>
+    <actuator name="left_wheel_back_motor">
+      <hardwareInterface>hardware_interface/EffortJointInterface</hardwareInterface>
+      <mechanicalReduction>1</mechanicalReduction>
+    </actuator>
+  </transmission>
+  <transmission name="left_wheel_front_tran">
+    <type>transmission_interface/SimpleTransmission</type>
+    <joint name="left_wheel_front_hinge">
+      <hardwareInterface>hardware_interface/EffortJointInterface</hardwareInterface>
+    </joint>
+    <actuator name="left_wheel_front_motor">
+      <hardwareInterface>hardware_interface/EffortJointInterface</hardwareInterface>
+      <mechanicalReduction>1</mechanicalReduction>
+    </actuator>
+  </transmission>
+  <transmission name="right_wheel_back_tran">
+    <type>transmission_interface/SimpleTransmission</type>
+    <joint name="right_wheel_back_hinge">
+      <hardwareInterface>hardware_interface/EffortJointInterface</hardwareInterface>
+    </joint>
+    <actuator name="right_wheel_back_motor">
+      <hardwareInterface>hardware_interface/EffortJointInterface</hardwareInterface>
+      <mechanicalReduction>1</mechanicalReduction>
+    </actuator>
+  </transmission>
+  <transmission name="right_wheel_front_tran">
+    <type>transmission_interface/SimpleTransmission</type>
+    <joint name="right_wheel_front_hinge">
+      <hardwareInterface>hardware_interface/EffortJointInterface</hardwareInterface>
+    </joint>
+    <actuator name="right_wheel_front_motor">
+      <hardwareInterface>hardware_interface/EffortJointInterface</hardwareInterface>
+      <mechanicalReduction>1</mechanicalReduction>
+    </actuator>
+  </transmission>
   <joint name="camera_joint" type="fixed">
     <axis xyz="0 1 0" />
-    <origin xyz=".47 .03 0" rpy="0 0 0"/>
-    <parent link="base_link"/>
-    <child link="f_stereo_1"/>
-  </joint>
-  <joint name="camera_joint2" type="fixed">
-    <axis xyz="0 1 0" />
-    <origin xyz=".47 -.03 0" rpy="0 0 0"/>
-    <parent link="base_link"/>
-    <child link="f_stereo_2"/>
-  </joint>
-  <joint name="camera_joint3" type="fixed">
-    <axis xyz="0 1 0" />
-    <origin xyz="-.47 .03 0" rpy="0 0 3.14"/>
-    <parent link="base_link"/>
-    <child link="f_stereo_3"/>
-  </joint>
-  <joint name="camera_joint4" type="fixed">
-    <axis xyz="0 1 0" />
-    <origin xyz="-.47 -.03 0" rpy="0 0 3.14"/>
-    <parent link="base_link"/>
-    <child link="f_stereo_4"/>
+    <origin xyz="0.1 0 0" rpy="0 0 0"/>
+    <parent link="drum_back"/>
+    <child link="camera_back"/>
   </joint>
   <joint type="continuous" name="left_wheel_front_hinge">
@@ -333,5 +247,5 @@
     <axis xyz="0 1 0" rpy="0 0 0"/>
     <limit effort="100" velocity="100"/>
-    <joint_properties damping="0.0" friction="0.0"/>
+    <joint_properties damping="0.1" friction="0.7"/>
   </joint>
   <joint type="continuous" name="right_wheel_front_hinge">
@@ -341,5 +255,5 @@
     <axis xyz="0 1 0" rpy="0 0 0"/>
     <limit effort="100" velocity="100"/>
-    <joint_properties damping="0.0" friction="0.0"/>
+    <joint_properties damping="0.1" friction="0.7"/>
   </joint>
   <joint type="continuous" name="left_wheel_back_hinge">
@@ -349,5 +263,5 @@
     <axis xyz="0 1 0" rpy="0 0 0"/>
     <limit effort="100" velocity="100"/>
-    <joint_properties damping="0.0" friction="0.0"/>
+    <joint_properties damping="0.1" friction="0.7"/>
   </joint>
   <joint type="continuous" name="right_wheel_back_hinge">
@@ -357,7 +271,7 @@
     <axis xyz="0 1 0" rpy="0 0 0"/>
     <limit effort="100" velocity="100"/>
-    <joint_properties damping="0.0" friction="0.0"/>
-  </joint>
-  <joint type="continuous" name="arm_back_hinge">
+    <joint_properties damping="0.1" friction="0.7"/>
+  </joint>
+  <joint type="fixed" name="arm_back_hinge">
     <origin xyz="-0.2 0 0" rpy="0 0 1.57"/>
     <child link="arm_back"/>
@@ -367,5 +281,5 @@
     <joint_properties damping="0.0" friction="0.0"/>
   </joint>
-  <joint type="continuous" name="arm_front_hinge">
+  <joint type="fixed" name="arm_front_hinge">
     <origin xyz="0.2 0 0" rpy="0 0 1.57"/>
     <child link="arm_front"/>
@@ -375,5 +289,5 @@
     <joint_properties damping="0.0" friction="0.0"/>
   </joint>
-  <joint type="continuous" name="drum_front_hinge">
+  <joint type="fixed" name="drum_front_hinge">
     <origin xyz="0 -0.2 0" rpy="0 0 1.57"/>
     <child link="drum_front"/>
@@ -383,5 +297,5 @@
     <joint_properties damping="0.0" friction="0.0"/>
   </joint>
-  <joint type="continuous" name="drum_back_hinge">
+  <joint type="fixed" name="drum_back_hinge">
     <origin xyz="0 0.2 0" rpy="0 0 1.57"/>
     <child link="drum_back"/>
