Commit message: Added controller support to Gazebo sim for driving.

File: packages/ai_swarm/ez_rassor_description/urdf/ez_rassor.xacro (robot description, xacro)
@@ -1,13 +1,20 @@
 <?xml version='1.0'?>
 <robot name="ez_rassor" xmlns:xacro="http://www.ros.org/wiki/xacro">
- <xacro:include filename="$(find ez_rassor_description)/urdf/ez_rassor.gazebo" />
- <xacro:include filename="$(find ez_rassor_description)/urdf/materials.xacro" />
- <xacro:include filename="$(find ez_rassor_description)/urdf/macros.xacro" />
+  <xacro:property name="cameraSize" value="0.05"/>
+  <xacro:property name="cameraMass" value="0.1"/>
+  <xacro:include filename="$(find ez_rassor_description)/urdf/ez_rassor.gazebo" />
+  <xacro:include filename="$(find ez_rassor_description)/urdf/materials.xacro" />
+  <xacro:include filename="$(find ez_rassor_description)/urdf/macros.xacro" />
+  <!--Below are all of the robot's Links/-->
   <link name='base_link'>
     <pose>0 0 0.1 0 0 0</pose>
     <inertial>
-      <mass value="1.0"/>
+      <mass value="10.0"/>
       <origin xyz="0.0 0 0.1" rpy=" 0 0 0"/>
-      <box_inertia m="1.0" x=".4" y=".2" z=".1"/>
+      <inertia
+          ixx="0.5" ixy="0" ixz="0"
+          iyy="1.0" iyz="0"
+          izz="0.1"
+      />
     </inertial>
     <collision name='collision'>
@@ -27,5 +34,5 @@
       <origin xyz="0 0 0" rpy="0 1.5707 1.5707"/>
       <geometry>
-          <mesh filename="package://ez_rassor_description/meshes/wheel.dae"/>
+        <cylinder radius="0.1" length="0.05"/>
       </geometry>
     </collision>
@@ -33,11 +40,15 @@
       <origin xyz="0 0 0" rpy="0 1.5707 1.5707"/>
       <geometry>
-          <mesh filename="package://ez_rassor_description/meshes/wheel.dae"/>
-      </geometry>
-    </visual>
-    <inertial>
-      <origin xyz="0 0 0" rpy="0 1.5707 1.5707"/>
-      <mass value=".5"/>
-      <cylinder_inertia m=".5" r="0.1" h="0.05"/>
+        <cylinder radius="0.1" length="0.05"/>
+      </geometry>
+    </visual>
+    <inertial>
+      <origin xyz="0 0 0" rpy="0 1.5707 1.5707"/>
+      <mass value="5"/>
+      <cylinder_inertia m="5" r="0.1" h="0.05"/>
+      <inertia
+        ixx="1.0" ixy="0.0" ixz="0.0"
+        iyy="1.0" iyz="0.0"
+        izz="1.0"/>
     </inertial>
   </link>
@@ -46,5 +57,5 @@
       <origin xyz="0 0 0" rpy="0 1.5707 1.5707"/>
       <geometry>
-          <mesh filename="package://ez_rassor_description/meshes/wheel.dae"/>
+        <cylinder radius="0.1" length="0.05"/>
       </geometry>
     </collision>
@@ -52,11 +63,15 @@
       <origin xyz="0 0 0" rpy="0 1.5707 1.5707"/>
       <geometry>
-          <mesh filename="package://ez_rassor_description/meshes/wheel.dae"/>
-      </geometry>
-    </visual>
-    <inertial>
-      <origin xyz="0 0 0" rpy="0 1.5707 1.5707"/>
-      <mass value=".5"/>
-      <cylinder_inertia m=".5" r="0.1" h="0.05"/>
+        <cylinder radius="0.1" length="0.05"/>
+      </geometry>
+    </visual>
+    <inertial>
+      <origin xyz="0 0 0" rpy="0 1.5707 1.5707"/>
+      <mass value="5"/>
+      <cylinder_inertia m="5" r="0.1" h="0.05"/>
+      <inertia
+        ixx="1.0" ixy="0.0" ixz="0.0"
+        iyy="1.0" iyz="0.0"
+        izz="1.0"/>
     </inertial>
   </link>
@@ -65,5 +80,5 @@
       <origin xyz="0 0 0" rpy="0 1.5707 1.5707"/>
       <geometry>
-          <mesh filename="package://ez_rassor_description/meshes/wheel.dae"/>
+        <cylinder radius="0.1" length="0.05"/>
       </geometry>
     </collision>
@@ -71,11 +86,15 @@
       <origin xyz="0 0 0" rpy="0 1.5707 1.5707"/>
       <geometry>
-          <mesh filename="package://ez_rassor_description/meshes/wheel.dae"/>
-      </geometry>
-    </visual>
-    <inertial>
-      <origin xyz="0 0 0" rpy="0 1.5707 1.5707"/>
-      <mass value=".5"/>
-      <cylinder_inertia m=".5" r="0.1" h="0.05"/>
+        <cylinder radius="0.1" length="0.05"/>
+      </geometry>
+    </visual>
+    <inertial>
+      <origin xyz="0 0 0" rpy="0 1.5707 1.5707"/>
+      <mass value="5"/>
+      <cylinder_inertia m="5" r="0.1" h="0.05"/>
+      <inertia
+        ixx="1.0" ixy="0.0" ixz="0.0"
+        iyy="1.0" iyz="0.0"
+        izz="1.0"/>
     </inertial>
   </link>
@@ -84,5 +103,5 @@
       <origin xyz="0 0 0" rpy="0 1.5707 1.5707"/>
       <geometry>
-          <mesh filename="package://ez_rassor_description/meshes/wheel.dae"/>
+        <cylinder radius="0.1" length="0.05"/>
       </geometry>
     </collision>
@@ -90,11 +109,15 @@
       <origin xyz="0 0 0" rpy="0 1.5707 1.5707"/>
       <geometry>
-          <mesh filename="package://ez_rassor_description/meshes/wheel.dae"/>
-      </geometry>
-    </visual>
-    <inertial>
-      <origin xyz="0 0 0" rpy="0 1.5707 1.5707"/>
-      <mass value=".5"/>
-      <cylinder_inertia m=".5" r="0.1" h="0.05"/>
+        <cylinder radius="0.1" length="0.05"/>
+      </geometry>
+    </visual>
+    <inertial>
+      <origin xyz="0 0 0" rpy="0 1.5707 1.5707"/>
+      <mass value="5"/>
+      <cylinder_inertia m="5" r="0.1" h="0.05"/>
+      <inertia
+        ixx="1.0" ixy="0.0" ixz="0.0"
+        iyy="1.0" iyz="0.0"
+        izz="1.0"/>
     </inertial>
   </link>
@@ -114,6 +137,10 @@
     <inertial>
       <origin xyz="0 0 0" rpy="0 1.5707 1.5707"/>
-      <mass value=".5"/>
-      <cylinder_inertia m=".5" r="0.1" h="0.05"/>
+      <mass value="5"/>
+      <cylinder_inertia m="5" r="0.1" h="0.05"/>
+      <inertia
+        ixx="1.0" ixy="0.0" ixz="0.0"
+        iyy="1.0" iyz="0.0"
+        izz="1.0"/>
     </inertial>
   </link>
@@ -133,6 +160,10 @@
     <inertial>
       <origin xyz="0 0 0" rpy="0 1.5707 1.5707"/>
-      <mass value=".5"/>
-      <cylinder_inertia m=".5" r="0.1" h="0.05"/>
+      <mass value="5"/>
+      <cylinder_inertia m="5" r="0.1" h="0.05"/>
+      <inertia
+        ixx="1.0" ixy="0.0" ixz="0.0"
+        iyy="1.0" iyz="0.0"
+        izz="1.0"/>
     </inertial>
   </link>
@@ -141,5 +172,5 @@
       <origin xyz="0 0 0" rpy="0 1.5707 1.5707"/>
       <geometry>
-        <cylinder radius="0.07" length="0.05"/>
+        <cylinder radius="0.08" length="0.05"/>
       </geometry>
     </collision>
@@ -152,6 +183,10 @@
     <inertial>
       <origin xyz="0 0 0" rpy="0 1.5707 1.5707"/>
-      <mass value="10"/>
-      <cylinder_inertia m="10" r="0.1" h="0.05"/>
+      <mass value="5"/>
+      <cylinder_inertia m="5" r="0.1" h="0.05"/>
+      <inertia
+        ixx="1.0" ixy="0.0" ixz="0.0"
+        iyy="1.0" iyz="0.0"
+        izz="1.0"/>
     </inertial>
   </link>
@@ -160,5 +195,5 @@
       <origin xyz="0 0 0" rpy="0 1.5707 1.5707"/>
       <geometry>
-        <cylinder radius="0.07" length="0.05"/>
+        <cylinder radius="0.08" length="0.05"/>
       </geometry>
     </collision>
@@ -171,35 +206,20 @@
     <inertial>
       <origin xyz="0 0 0" rpy="0 1.5707 1.5707"/>
-      <mass value="10"/>
-      <cylinder_inertia m="10" r="0.1" h="0.05"/>
-    </inertial>
-  </link>
-  <link name="camera_back">
-    <collision>
-      <origin xyz="0 0 0" rpy="0 1.57 1.57"/>
-      <geometry>
-    <box size=".1 .1 .1"/>
-      </geometry>
-    </collision>
-    <visual>
-      <origin xyz="0 0 0" rpy="0 0 0"/>
-      <geometry>
-    <box size=".1 .1 .1"/>
-      </geometry>
-      <material name="red"/>
-    </visual>
-    <inertial>
-      <mass value="1e-5" />
-      <origin xyz="0 0 0" rpy="0 0 0"/>
-      <box_inertia m="1e-5" x=".1" y = ".1" z=".1"/>
-    </inertial>
-  </link>
-  <transmission name="left_wheel_back_tran">
+      <mass value="5"/>
+      <cylinder_inertia m="5" r="0.1" h="0.05"/>
+      <inertia
+        ixx="1.0" ixy="0.0" ixz="0.0"
+        iyy="1.0" iyz="0.0"
+        izz="1.0"/>
+    </inertial>
+  </link>
+<!-- Transmissions -->
+<transmission name="left_wheel_back_tran">
     <type>transmission_interface/SimpleTransmission</type>
     <joint name="left_wheel_back_hinge">
-      <hardwareInterface>hardware_interface/EffortJointInterface</hardwareInterface>
+      <hardwareInterface>hardware_interface/VelocityJointInterface</hardwareInterface>
     </joint>
     <actuator name="left_wheel_back_motor">
-      <hardwareInterface>hardware_interface/EffortJointInterface</hardwareInterface>
+      <hardwareInterface>hardware_interface/VelocityJointInterface</hardwareInterface>
       <mechanicalReduction>1</mechanicalReduction>
     </actuator>
@@ -208,8 +228,8 @@
     <type>transmission_interface/SimpleTransmission</type>
     <joint name="left_wheel_front_hinge">
-      <hardwareInterface>hardware_interface/EffortJointInterface</hardwareInterface>
+      <hardwareInterface>hardware_interface/VelocityJointInterface</hardwareInterface>
     </joint>
     <actuator name="left_wheel_front_motor">
-      <hardwareInterface>hardware_interface/EffortJointInterface</hardwareInterface>
+      <hardwareInterface>hardware_interface/VelocityJointInterface</hardwareInterface>
       <mechanicalReduction>1</mechanicalReduction>
     </actuator>
@@ -218,8 +238,8 @@
     <type>transmission_interface/SimpleTransmission</type>
     <joint name="right_wheel_back_hinge">
-      <hardwareInterface>hardware_interface/EffortJointInterface</hardwareInterface>
+      <hardwareInterface>hardware_interface/VelocityJointInterface</hardwareInterface>
     </joint>
     <actuator name="right_wheel_back_motor">
-      <hardwareInterface>hardware_interface/EffortJointInterface</hardwareInterface>
+      <hardwareInterface>hardware_interface/VelocityJointInterface</hardwareInterface>
       <mechanicalReduction>1</mechanicalReduction>
     </actuator>
@@ -228,16 +248,123 @@
     <type>transmission_interface/SimpleTransmission</type>
     <joint name="right_wheel_front_hinge">
-      <hardwareInterface>hardware_interface/EffortJointInterface</hardwareInterface>
+      <hardwareInterface>hardware_interface/VelocityJointInterface</hardwareInterface>
     </joint>
     <actuator name="right_wheel_front_motor">
-      <hardwareInterface>hardware_interface/EffortJointInterface</hardwareInterface>
+      <hardwareInterface>hardware_interface/VelocityJointInterface</hardwareInterface>
       <mechanicalReduction>1</mechanicalReduction>
     </actuator>
   </transmission>
+  <!--First Camera Added/-->
+  <link name="f_stereo_1">
+    <collision>
+      <origin xyz="0 0 0" rpy="0 0 0"/>
+      <geometry>
+        <box size="${cameraSize} ${cameraSize} ${cameraSize}"/>
+      </geometry>
+    </collision>
+    <visual>
+      <origin xyz="0 0 0" rpy="0 0 0"/>
+      <geometry>
+        <box size="${cameraSize} ${cameraSize} ${cameraSize}"/>
+      </geometry>
+      <material name="green"/>
+    </visual>
+    <inertial>
+      <mass value="${cameraMass}" />
+      <origin xyz="0 0 0" rpy="0 0 0"/>
+      <box_inertia m="${cameraMass}" x="${cameraSize}" y="${cameraSize}" z="${cameraSize}" />
+      <inertia ixx="1e-6" ixy="0" ixz="0" iyy="1e-6" iyz="0" izz="1e-6" />
+    </inertial>
+  </link>
+  <!--Second Camera Added/-->
+  <link name="f_stereo_2">
+    <collision>
+      <origin xyz="0 0 0" rpy="0 0 0"/>
+      <geometry>
+        <box size="${cameraSize} ${cameraSize} ${cameraSize}"/>
+      </geometry>
+    </collision>
+    <visual>
+      <origin xyz="0 0 0" rpy="0 0 0"/>
+      <geometry>
+        <box size="${cameraSize} ${cameraSize} ${cameraSize}"/>
+      </geometry>
+      <material name="green"/>
+    </visual>
+    <inertial>
+      <mass value="${cameraMass}" />
+      <origin xyz="0 0 0" rpy="0 0 0"/>
+      <box_inertia m="${cameraMass}" x="${cameraSize}" y="${cameraSize}" z="${cameraSize}" />
+      <inertia ixx="1e-6" ixy="0" ixz="0" iyy="1e-6" iyz="0" izz="1e-6" />
+    </inertial>
+  </link>
+    <!--Third Camera Added/-->
+  <link name="f_stereo_3">
+    <collision>
+      <origin xyz="0 0 0" rpy="0 0 0"/>
+      <geometry>
+        <box size="${cameraSize} ${cameraSize} ${cameraSize}"/>
+      </geometry>
+    </collision>
+    <visual>
+      <origin xyz="0 0 0" rpy="0 0 0"/>
+      <geometry>
+        <box size="${cameraSize} ${cameraSize} ${cameraSize}"/>
+      </geometry>
+      <material name="green"/>
+    </visual>
+    <inertial>
+      <mass value="${cameraMass}" />
+      <origin xyz="0 0 0" rpy="0 0 0"/>
+      <box_inertia m="${cameraMass}" x="${cameraSize}" y="${cameraSize}" z="${cameraSize}" />
+      <inertia ixx="1e-6" ixy="0" ixz="0" iyy="1e-6" iyz="0" izz="1e-6" />
+    </inertial>
+  </link>
+      <!--Fourth Camera Added/-->
+  <link name="f_stereo_4">
+    <collision>
+      <origin xyz="0 0 0" rpy="0 0 0"/>
+      <geometry>
+        <box size="${cameraSize} ${cameraSize} ${cameraSize}"/>
+      </geometry>
+    </collision>
+    <visual>
+      <origin xyz="0 0 0" rpy="0 0 0"/>
+      <geometry>
+        <box size="${cameraSize} ${cameraSize} ${cameraSize}"/>
+      </geometry>
+      <material name="green"/>
+    </visual>
+    <inertial>
+      <mass value="${cameraMass}" />
+      <origin xyz="0 0 0" rpy="0 0 0"/>
+      <box_inertia m="${cameraMass}" x="${cameraSize}" y="${cameraSize}" z="${cameraSize}" />
+      <inertia ixx="1e-6" ixy="0" ixz="0" iyy="1e-6" iyz="0" izz="1e-6" />
+    </inertial>
+  </link>
+  <!--Below are all of the robot's joints/-->
   <joint name="camera_joint" type="fixed">
     <axis xyz="0 1 0" />
-    <origin xyz="0.1 0 0" rpy="0 0 0"/>
-    <parent link="drum_back"/>
-    <child link="camera_back"/>
+    <origin xyz=".47 .03 0" rpy="0 0 0"/>
+    <parent link="base_link"/>
+    <child link="f_stereo_1"/>
+  </joint>
+  <joint name="camera_joint2" type="fixed">
+    <axis xyz="0 1 0" />
+    <origin xyz=".47 -.03 0" rpy="0 0 0"/>
+    <parent link="base_link"/>
+    <child link="f_stereo_2"/>
+  </joint>
+  <joint name="camera_joint3" type="fixed">
+    <axis xyz="0 1 0" />
+    <origin xyz="-.47 .03 0" rpy="0 0 3.14"/>
+    <parent link="base_link"/>
+    <child link="f_stereo_3"/>
+  </joint>
+  <joint name="camera_joint4" type="fixed">
+    <axis xyz="0 1 0" />
+    <origin xyz="-.47 -.03 0" rpy="0 0 3.14"/>
+    <parent link="base_link"/>
+    <child link="f_stereo_4"/>
   </joint>
   <joint type="continuous" name="left_wheel_front_hinge">
@@ -247,5 +374,5 @@
     <axis xyz="0 1 0" rpy="0 0 0"/>
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
Commit message: Added controller support to Gazebo sim for arm movement.

File: packages/ai_swarm/ez_rassor_description/urdf/ez_rassor.xacro (robot description, xacro)
@@ -255,4 +255,24 @@
     </actuator>
   </transmission>
+  <transmission name="arm_front_tran">
+    <type>transmission_interface/SimpleTransmission</type>
+    <joint name="arm_front_hinge">
+      <hardwareInterface>hardware_interface/VelocityJointInterface</hardwareInterface>
+    </joint>
+    <actuator name="arm_front_motor">
+      <hardwareInterface>hardware_interface/VelocityJointInterface</hardwareInterface>
+      <mechanicalReduction>1</mechanicalReduction>
+    </actuator>
+  </transmission>
+  <transmission name="arm_back_tran">
+    <type>transmission_interface/SimpleTransmission</type>
+    <joint name="arm_back_hinge">
+      <hardwareInterface>hardware_interface/VelocityJointInterface</hardwareInterface>
+    </joint>
+    <actuator name="arm_back_motor">
+      <hardwareInterface>hardware_interface/VelocityJointInterface</hardwareInterface>
+      <mechanicalReduction>1</mechanicalReduction>
+    </actuator>
+  </transmission>
   <!--First Camera Added/-->
   <link name="f_stereo_1">
@@ -400,5 +420,5 @@
     <joint_properties damping="0.0" friction="0.0"/>
   </joint>
-  <joint type="fixed" name="arm_back_hinge">
+  <joint type="continuous" name="arm_back_hinge">
     <origin xyz="-0.2 0 0" rpy="0 0 1.57"/>
     <child link="arm_back"/>
@@ -408,5 +428,5 @@
     <joint_properties damping="0.0" friction="0.0"/>
   </joint>
-  <joint type="fixed" name="arm_front_hinge">
+  <joint type="continuous" name="arm_front_hinge">
     <origin xyz="0.2 0 0" rpy="0 0 1.57"/>
     <child link="arm_front"/>

Commit message: Update ez_rassor.xacro
Shrink the visible size of all cameras

File: packages/ai_swarm/ez_rassor_description/urdf/ez_rassor.xacro (robot description, xacro)
@@ -1,5 +1,5 @@
 <?xml version='1.0'?>
 <robot name="ez_rassor" xmlns:xacro="http://www.ros.org/wiki/xacro">
-  <xacro:property name="cameraSize" value="0.05"/>
+  <xacro:property name="cameraSize" value="0.005"/>
   <xacro:property name="cameraMass" value="0.1"/>
   <xacro:include filename="$(find ez_rassor_description)/urdf/ez_rassor.gazebo" />

Commit message: Added IMU

File: packages/ai_swarm/ez_rassor_description/urdf/ez_rassor.xacro (robot description, xacro)
@@ -363,4 +363,26 @@
     </inertial>
   </link>
+  <!-- IMU -->
+  <link name="imu_link">
+    <collision>
+      <origin xyz="0 0 0" rpy="0 0 0"/>
+      <geometry>
+        <box size="${cameraSize} ${cameraSize} ${cameraSize}"/>
+      </geometry>
+    </collision>
+    <visual>
+      <origin xyz="0 0 0" rpy="0 0 0"/>
+      <geometry>
+        <box size="${cameraSize} ${cameraSize} ${cameraSize}"/>
+      </geometry>
+      <material name="green"/>
+    </visual>
+    <inertial>
+      <mass value="${cameraMass}" />
+      <origin xyz="0 0 0" rpy="0 0 0"/>
+      <box_inertia m="${cameraMass}" x="${cameraSize}" y="${cameraSize}" z="${cameraSize}" />
+      <inertia ixx="1e-6" ixy="0" ixz="0" iyy="1e-6" iyz="0" izz="1e-6" />
+    </inertial>
+  </link>
   <!--Below are all of the robot's joints/-->
   <joint name="camera_joint" type="fixed">
@@ -388,4 +410,10 @@
     <child link="f_stereo_4"/>
   </joint>
+  <joint name="imu_joint" type="fixed">
+    <axis xyz="0 0 0" />
+    <origin xyz="0 0 0" rpy="0 0 0"/>
+    <parent link="base_link"/>
+    <child link="imu_link"/>
+  </joint>
   <joint type="continuous" name="left_wheel_front_hinge">
     <origin xyz="0.15 0.15 0" rpy="0 0 0"/>

Commit message: Added IMU

File: packages/ai_swarm/ez_rassor_description/urdf/ez_rassor.xacro (robot description, xacro)
@@ -363,5 +363,5 @@
     </inertial>
   </link>
-  <!-- IMU -->
+    <!-- IMU -->
   <link name="imu_link">
     <collision>
@@ -385,4 +385,10 @@
     </inertial>
   </link>
+  <joint name="imu_joint" type="fixed">
+    <axis xyz="0 0 0" />
+    <origin xyz="0 0 0" rpy="0 0 0"/>
+    <parent link="base_link"/>
+    <child link="imu_link"/>
+  </joint>
   <!--Below are all of the robot's joints/-->
   <joint name="camera_joint" type="fixed">
@@ -410,10 +416,4 @@
     <child link="f_stereo_4"/>
   </joint>
-  <joint name="imu_joint" type="fixed">
-    <axis xyz="0 0 0" />
-    <origin xyz="0 0 0" rpy="0 0 0"/>
-    <parent link="base_link"/>
-    <child link="imu_link"/>
-  </joint>
   <joint type="continuous" name="left_wheel_front_hinge">
     <origin xyz="0.15 0.15 0" rpy="0 0 0"/>

Commit message: Fixed Cameras to have proper stereo settings

File: packages/ai_swarm/ez_rassor_description/urdf/ez_rassor.xacro (robot description, xacro)
@@ -275,72 +275,6 @@
     </actuator>
   </transmission>
-  <!--First Camera Added/-->
-  <link name="f_stereo_1">
-    <collision>
-      <origin xyz="0 0 0" rpy="0 0 0"/>
-      <geometry>
-        <box size="${cameraSize} ${cameraSize} ${cameraSize}"/>
-      </geometry>
-    </collision>
-    <visual>
-      <origin xyz="0 0 0" rpy="0 0 0"/>
-      <geometry>
-        <box size="${cameraSize} ${cameraSize} ${cameraSize}"/>
-      </geometry>
-      <material name="green"/>
-    </visual>
-    <inertial>
-      <mass value="${cameraMass}" />
-      <origin xyz="0 0 0" rpy="0 0 0"/>
-      <box_inertia m="${cameraMass}" x="${cameraSize}" y="${cameraSize}" z="${cameraSize}" />
-      <inertia ixx="1e-6" ixy="0" ixz="0" iyy="1e-6" iyz="0" izz="1e-6" />
-    </inertial>
-  </link>
-  <!--Second Camera Added/-->
-  <link name="f_stereo_2">
-    <collision>
-      <origin xyz="0 0 0" rpy="0 0 0"/>
-      <geometry>
-        <box size="${cameraSize} ${cameraSize} ${cameraSize}"/>
-      </geometry>
-    </collision>
-    <visual>
-      <origin xyz="0 0 0" rpy="0 0 0"/>
-      <geometry>
-        <box size="${cameraSize} ${cameraSize} ${cameraSize}"/>
-      </geometry>
-      <material name="green"/>
-    </visual>
-    <inertial>
-      <mass value="${cameraMass}" />
-      <origin xyz="0 0 0" rpy="0 0 0"/>
-      <box_inertia m="${cameraMass}" x="${cameraSize}" y="${cameraSize}" z="${cameraSize}" />
-      <inertia ixx="1e-6" ixy="0" ixz="0" iyy="1e-6" iyz="0" izz="1e-6" />
-    </inertial>
-  </link>
-    <!--Third Camera Added/-->
-  <link name="f_stereo_3">
-    <collision>
-      <origin xyz="0 0 0" rpy="0 0 0"/>
-      <geometry>
-        <box size="${cameraSize} ${cameraSize} ${cameraSize}"/>
-      </geometry>
-    </collision>
-    <visual>
-      <origin xyz="0 0 0" rpy="0 0 0"/>
-      <geometry>
-        <box size="${cameraSize} ${cameraSize} ${cameraSize}"/>
-      </geometry>
-      <material name="green"/>
-    </visual>
-    <inertial>
-      <mass value="${cameraMass}" />
-      <origin xyz="0 0 0" rpy="0 0 0"/>
-      <box_inertia m="${cameraMass}" x="${cameraSize}" y="${cameraSize}" z="${cameraSize}" />
-      <inertia ixx="1e-6" ixy="0" ixz="0" iyy="1e-6" iyz="0" izz="1e-6" />
-    </inertial>
-  </link>
-      <!--Fourth Camera Added/-->
-  <link name="f_stereo_4">
+  <!--Front Camera Added/-->
+  <link name="stereo_camera_front">
     <collision>
       <origin xyz="0 0 0" rpy="0 0 0"/>
@@ -392,27 +326,9 @@
   </joint>
   <!--Below are all of the robot's joints/-->
-  <joint name="camera_joint" type="fixed">
+  <joint name="front_camera_joint" type="fixed">
     <axis xyz="0 1 0" />
     <origin xyz=".47 .03 0" rpy="0 0 0"/>
     <parent link="base_link"/>
-    <child link="f_stereo_1"/>
-  </joint>
-  <joint name="camera_joint2" type="fixed">
-    <axis xyz="0 1 0" />
-    <origin xyz=".47 -.03 0" rpy="0 0 0"/>
-    <parent link="base_link"/>
-    <child link="f_stereo_2"/>
-  </joint>
-  <joint name="camera_joint3" type="fixed">
-    <axis xyz="0 1 0" />
-    <origin xyz="-.47 .03 0" rpy="0 0 3.14"/>
-    <parent link="base_link"/>
-    <child link="f_stereo_3"/>
-  </joint>
-  <joint name="camera_joint4" type="fixed">
-    <axis xyz="0 1 0" />
-    <origin xyz="-.47 -.03 0" rpy="0 0 3.14"/>
-    <parent link="base_link"/>
-    <child link="f_stereo_4"/>
+    <child link="stereo_camera_front"/>
   </joint>
   <joint type="continuous" name="left_wheel_front_hinge">
