Commit message: Fixed cameras more

File: packages/ai_swarm/ez_rassor_description/urdf/ez_rassor.xacro (robot description, xacro)
@@ -297,4 +297,26 @@
     </inertial>
   </link>
+<!--Back Camera Added/-->
+  <link name="stereo_camera_back">
+    <collision>
+      <origin xyz="0 0 0" rpy="0 0 0"/>
+      <geometry>
+        <box size="${cameraSize} ${cameraSize} ${cameraSize}"/>
+      </geometry>
+    </collision>
+    <visual>
+      <origin xyz="0 0 0" rpy="0 0 0"/>
+      <geometry>
+        <box size="${cameraSize} ${cameraSize} ${cameraSize}"/>
+      </geometry>
+      <material name="green"/>
+    </visual>
+    <inertial>
+      <mass value="${cameraMass}" />
+      <origin xyz="0 0 0" rpy="0 0 0"/>
+      <box_inertia m="${cameraMass}" x="${cameraSize}" y="${cameraSize}" z="${cameraSize}" />
+      <inertia ixx="1e-6" ixy="0" ixz="0" iyy="1e-6" iyz="0" izz="1e-6" />
+    </inertial>
+  </link>
     <!-- IMU -->
   <link name="imu_link">
@@ -326,9 +348,15 @@
   </joint>
   <!--Below are all of the robot's joints/-->
-  <joint name="front_camera_joint" type="fixed">
+  <joint name="camera_front_joint" type="fixed">
     <axis xyz="0 1 0" />
-    <origin xyz=".47 .03 0" rpy="0 0 0"/>
+    <origin xyz=".47 0 0" rpy="0 0 0"/>
     <parent link="base_link"/>
     <child link="stereo_camera_front"/>
+  </joint>
+  <joint name="camera_back_joint" type="fixed">
+    <axis xyz="0 1 0" />
+    <origin xyz="-.47 0 0" rpy="0 0 3.14"/>
+    <parent link="base_link"/>
+    <child link="stereo_camera_back"/>
   </joint>
   <joint type="continuous" name="left_wheel_front_hinge">

Commit message: Added custom drum arm and drums to model.

File: packages/ai_swarm/ez_rassor_description/urdf/ez_rassor.xacro (robot description, xacro)
@@ -32,86 +32,86 @@
   <link name="left_wheel_front">
     <collision name="collision">
+      <origin xyz="0 -0.06 0" rpy="3.14159 1.57079 -1.57089"/>
+      <geometry>
+        <robot_wheel />
+      </geometry>
+    </collision>
+    <visual name="left_wheel_front_visual">
+      <origin xyz="0 -0.06 0" rpy="-3.12268 1.57079 -1.55198"/>
+      <geometry>
+        <robot_wheel />
+      </geometry>
+    </visual>
+    <inertial>
+      <origin xyz="0 0 0" rpy="0 1.5707 1.5707" />
+      <mass value="5"/>
+      <cylinder_inertia m="5" r="0.1" h="0.05"/>
+      <inertia
+        ixx="1.0" ixy="0.0" ixz="0.0"
+        iyy="1.0" iyz="0.0"
+        izz="1.0"/>
+    </inertial>
+  </link>
+  <link name="right_wheel_front">
+    <collision name="collision">
+      <origin xyz="0 0.06 0" rpy="0 1.57079 -1.57089"/>
+      <geometry>
+        <robot_wheel />
+      </geometry>
+    </collision>
+    <visual name="right_wheel_front_visual">
+      <origin xyz="0 0.06 0" rpy="-0.00702 1.57079 -1.57316"/>
+      <geometry>
+        <robot_wheel />
+      </geometry>
+    </visual>
+    <inertial>
+      <origin rpy="0 1.5707 1.5707" xyz="0 0 0"/>
+      <mass value="5"/>
+      <cylinder_inertia m="5" r="0.1" h="0.05"/>
+      <inertia
+        ixx="1.0" ixy="0.0" ixz="0.0"
+        iyy="1.0" iyz="0.0"
+        izz="1.0"/>
+    </inertial>
+  </link>
+  <link name="left_wheel_back">
+    <collision name="collision">
+      <origin xyz="0 -0.06 0" rpy="3.14159  1.57079 -1.57089"/>
+      <geometry>
+        <robot_wheel />
+      </geometry>
+    </collision>
+    <visual name="left_wheel_back_visual">
+      <origin xyz="0 -0.06 0" rpy="-3.12268  1.57079 -1.55198"/>
+      <geometry>
+        <robot_wheel />
+      </geometry>
+    </visual>
+    <inertial>
       <origin xyz="0 0 0" rpy="0 1.5707 1.5707"/>
-      <geometry>
-        <cylinder radius="0.1" length="0.05"/>
-      </geometry>
-    </collision>
-    <visual name="left_wheel_front_visual">
+      <mass value="5"/>
+      <cylinder_inertia m="5" r="0.1" h="0.05"/>
+      <inertia
+        ixx="1.0" ixy="0.0" ixz="0.0"
+        iyy="1.0" iyz="0.0"
+        izz="1.0"/>
+    </inertial>
+  </link>
+  <link name="right_wheel_back">
+    <collision name="collision">
+      <origin xyz="0 0.06 0" rpy="0 1.57079 -1.57089"/>
+      <geometry>
+        <robot_wheel />
+      </geometry>
+    </collision>
+    <visual name="right_wheel_back_visual">
+      <origin xyz="0 0.06 0" rpy="-0.00702 1.57079 -1.57316"/>
+      <geometry>
+        <robot_wheel />
+      </geometry>
+    </visual>
+    <inertial>
       <origin xyz="0 0 0" rpy="0 1.5707 1.5707"/>
-      <geometry>
-        <cylinder radius="0.1" length="0.05"/>
-      </geometry>
-    </visual>
-    <inertial>
-      <origin xyz="0 0 0" rpy="0 1.5707 1.5707"/>
-      <mass value="5"/>
-      <cylinder_inertia m="5" r="0.1" h="0.05"/>
-      <inertia
-        ixx="1.0" ixy="0.0" ixz="0.0"
-        iyy="1.0" iyz="0.0"
-        izz="1.0"/>
-    </inertial>
-  </link>
-  <link name="right_wheel_front">
-    <collision name="collision">
-      <origin xyz="0 0 0" rpy="0 1.5707 1.5707"/>
-      <geometry>
-        <cylinder radius="0.1" length="0.05"/>
-      </geometry>
-    </collision>
-    <visual name="right_wheel_front_visual">
-      <origin xyz="0 0 0" rpy="0 1.5707 1.5707"/>
-      <geometry>
-        <cylinder radius="0.1" length="0.05"/>
-      </geometry>
-    </visual>
-    <inertial>
-      <origin xyz="0 0 0" rpy="0 1.5707 1.5707"/>
-      <mass value="5"/>
-      <cylinder_inertia m="5" r="0.1" h="0.05"/>
-      <inertia
-        ixx="1.0" ixy="0.0" ixz="0.0"
-        iyy="1.0" iyz="0.0"
-        izz="1.0"/>
-    </inertial>
-  </link>
-  <link name="left_wheel_back">
-    <collision name="collision">
-      <origin xyz="0 0 0" rpy="0 1.5707 1.5707"/>
-      <geometry>
-        <cylinder radius="0.1" length="0.05"/>
-      </geometry>
-    </collision>
-    <visual name="left_wheel_back_visual">
-      <origin xyz="0 0 0" rpy="0 1.5707 1.5707"/>
-      <geometry>
-        <cylinder radius="0.1" length="0.05"/>
-      </geometry>
-    </visual>
-    <inertial>
-      <origin xyz="0 0 0" rpy="0 1.5707 1.5707"/>
-      <mass value="5"/>
-      <cylinder_inertia m="5" r="0.1" h="0.05"/>
-      <inertia
-        ixx="1.0" ixy="0.0" ixz="0.0"
-        iyy="1.0" iyz="0.0"
-        izz="1.0"/>
-    </inertial>
-  </link>
-  <link name="right_wheel_back">
-    <collision name="collision">
-      <origin xyz="0 0 0" rpy="0 1.5707 1.5707"/>
-      <geometry>
-        <cylinder radius="0.1" length="0.05"/>
-      </geometry>
-    </collision>
-    <visual name="right_wheel_back_visual">
-      <origin xyz="0 0 0" rpy="0 1.5707 1.5707"/>
-      <geometry>
-        <cylinder radius="0.1" length="0.05"/>
-      </geometry>
-    </visual>
-    <inertial>
-      <origin xyz="0 0 0" rpy="0 1.5707 1.5707"/>
       <mass value="5"/>
       <cylinder_inertia m="5" r="0.1" h="0.05"/>
@@ -124,17 +124,17 @@
   <link name="arm_back">
     <collision name="collision">
-      <origin xyz="0 .1 0" rpy="0 1.5707 1.5707"/>
-      <geometry>
-        <cylinder radius="0.025" length="0.3"/>
-      </geometry>
-    </collision>
-    <visual name="arm_back_visual">
-      <origin xyz="0 .1 0" rpy="0 1.5707 1.5707"/>
-      <geometry>
-        <cylinder radius="0.025" length="0.3"/>
-      </geometry>
-    </visual>
-    <inertial>
-      <origin xyz="0 0 0" rpy="0 1.5707 1.5707"/>
+      <origin rpy="0 0 3.1415" xyz="0 0 0"/>
+      <geometry>
+        <robot_arm />
+      </geometry>
+    </collision>
+    <visual name="visual">
+      <origin rpy="0 0 3.1415" xyz="0 0 0"/>
+      <geometry>
+        <robot_arm />
+      </geometry>
+    </visual>
+    <inertial>
+      <origin xyz="0 0 0" rpy="0 0 3.1415"/>
       <mass value="5"/>
       <cylinder_inertia m="5" r="0.1" h="0.05"/>
@@ -147,17 +147,17 @@
   <link name="arm_front">
     <collision name="collision">
-      <origin xyz="0 -.1 0" rpy="0 1.5707 1.5707"/>
-      <geometry>
-        <cylinder radius="0.025" length="0.3"/>
-      </geometry>
-    </collision>
-    <visual name="arm_front_visual">
-      <origin xyz="0 -.1 0" rpy="0 1.5707 1.5707"/>
-      <geometry>
-        <cylinder radius="0.025" length="0.3"/>
-      </geometry>
-    </visual>
-    <inertial>
-      <origin xyz="0 0 0" rpy="0 1.5707 1.5707"/>
+      <origin rpy="0 0 0" xyz="0 0 0"/>
+      <geometry>
+        <robot_arm />
+      </geometry>
+    </collision>
+    <visual name="visual">
+      <origin rpy="0 0 0" xyz="0 0 0"/>
+      <geometry>
+        <robot_arm />
+      </geometry>
+    </visual>
+    <inertial>
+      <origin xyz="0 0 0" rpy="0 0 0"/>
       <mass value="5"/>
       <cylinder_inertia m="5" r="0.1" h="0.05"/>
@@ -170,17 +170,17 @@
   <link name="drum_front">
     <collision name="collision">
-      <origin xyz="0 0 0" rpy="0 1.5707 1.5707"/>
-      <geometry>
-        <cylinder radius="0.08" length="0.05"/>
+      <origin xyz="0 0 0" rpy="0 0 1.5707"/>
+      <geometry>
+        <robot_arm_drum />
       </geometry>
     </collision>
     <visual name="drum_front_visual">
-      <origin xyz="0 0 0" rpy="0 1.5707 1.5707"/>
-      <geometry>
-        <cylinder radius="0.08" length="0.4"/>
-      </geometry>
-    </visual>
-    <inertial>
-      <origin xyz="0 0 0" rpy="0 1.5707 1.5707"/>
+      <origin xyz="0 0 0" rpy="0 0 1.5707"/>
+      <geometry>
+        <robot_arm_drum />
+      </geometry>
+    </visual>
+    <inertial>
+      <origin xyz="0 0 0" rpy="0 0 1.5707"/>
       <mass value="5"/>
       <cylinder_inertia m="5" r="0.1" h="0.05"/>
@@ -193,17 +193,17 @@
   <link name="drum_back">
     <collision name="collision">
-      <origin xyz="0 0 0" rpy="0 1.5707 1.5707"/>
-      <geometry>
-        <cylinder radius="0.08" length="0.05"/>
+      <origin xyz="0 0 0" rpy="0 0 4.7122"/>
+      <geometry>
+        <robot_arm_drum />
       </geometry>
     </collision>
     <visual name="drum_back">
-      <origin xyz="0 0 0" rpy="0 1.5707 1.5707"/>
-      <geometry>
-        <cylinder radius="0.08" length="0.4"/>
-      </geometry>
-    </visual>
-    <inertial>
-      <origin xyz="0 0 0" rpy="0 1.5707 1.5707"/>
+      <origin xyz="0 0 0" rpy="0 0 4.7122"/>
+      <geometry>
+        <robot_arm_drum />
+      </geometry>
+    </visual>
+    <inertial>
+      <origin xyz="0 0 0" rpy="0 0 4.7122"/>
       <mass value="5"/>
       <cylinder_inertia m="5" r="0.1" h="0.05"/>
@@ -449,21 +449,21 @@
   </joint>
   <joint type="continuous" name="arm_back_hinge">
-    <origin xyz="-0.2 0 0" rpy="0 0 1.57"/>
+    <origin xyz="-0.25 0 0" rpy="0 0 6.2828"/>
     <child link="arm_back"/>
     <parent link="base_link"/>
-    <axis xyz="1 0 0" rpy="0 0 0"/>
+    <axis xyz="0 1 0" rpy="0 0 0"/>
     <limit effort="100" velocity="100"/>
     <joint_properties damping="0.0" friction="0.0"/>
   </joint>
   <joint type="continuous" name="arm_front_hinge">
-    <origin xyz="0.2 0 0" rpy="0 0 1.57"/>
+    <origin xyz="0.25 0 0" rpy="0 0 6.2828"/>
     <child link="arm_front"/>
     <parent link="base_link"/>
-    <axis xyz="1 0 0" rpy="0 0 0"/>
+    <axis xyz="0 1 0" rpy="0 0 0"/>
     <limit effort="100" velocity="100"/>
     <joint_properties damping="0.0" friction="0.0"/>
   </joint>
   <joint type="continuous" name="drum_front_hinge">
-    <origin xyz="0 -0.2 0" rpy="0 0 1.57"/>
+    <origin xyz="0.338245 0 0" rpy="0 0 6.2828"/>
     <child link="drum_front"/>
     <parent link="arm_front"/>
@@ -473,5 +473,5 @@
   </joint>
   <joint type="continuous" name="drum_back_hinge">
-    <origin xyz="0 0.2 0" rpy="0 0 1.57"/>
+    <origin xyz="-0.338245 0 0" rpy="0 0 6.2828"/>
     <child link="drum_back"/>
     <parent link="arm_back"/>

File: packages/ai_swarm/ez_rassor_description/urdf/macros.xacro (robot description, xacro)
@@ -19,3 +19,12 @@
     />
     </macro>
+    <macro name="robot_arm">
+        <mesh filename="package://ez_rassor_description/meshes/drum_arm_short.dae" scale="1.0 1.0 1.0"></mesh>
+    </macro>
+    <macro name="robot_arm_drum">
+        <mesh filename="package://ez_rassor_description/meshes/drum.dae" scale="1.5 1.5 1.5"></mesh>
+    </macro>
+    <macro name="robot_wheel">
+        <mesh filename="package://ez_rassor_description/meshes/wheel.dae" scale="1.1 1.1 1.1"></mesh>
+    </macro>
 </robot>

Commit message: Tiny extra fixes for camera

File: packages/ai_swarm/ez_rassor_description/urdf/ez_rassor.xacro (robot description, xacro)
@@ -350,5 +350,5 @@
   <joint name="camera_front_joint" type="fixed">
     <axis xyz="0 1 0" />
-    <origin xyz=".47 0 0" rpy="0 0 0"/>
+    <origin xyz=".75 0 0" rpy="0 0 0"/>
     <parent link="base_link"/>
     <child link="stereo_camera_front"/>
@@ -356,5 +356,5 @@
   <joint name="camera_back_joint" type="fixed">
     <axis xyz="0 1 0" />
-    <origin xyz="-.47 0 0" rpy="0 0 3.14"/>
+    <origin xyz="-.75 0 0" rpy="0 0 3.14"/>
     <parent link="base_link"/>
     <child link="stereo_camera_back"/>

Commit message: Fixed round two

File: packages/ai_swarm/ez_rassor_description/urdf/ez_rassor.xacro (robot description, xacro)
@@ -1,9 +1,5 @@
 <?xml version='1.0'?>
 <robot name="ez_rassor" xmlns:xacro="http://www.ros.org/wiki/xacro">
-<<<<<<< HEAD
   <xacro:property name="cameraSize" value="0.005"/>
-=======
-  <xacro:property name="cameraSize" value="0.05"/>
->>>>>>> master
   <xacro:property name="cameraMass" value="0.1"/>
   <xacro:include filename="$(find ez_rassor_description)/urdf/ez_rassor.gazebo" />
@@ -48,9 +44,5 @@
     </visual>
     <inertial>
-<<<<<<< HEAD
       <origin xyz="0 0 0" rpy="0 1.5707 1.5707" />
-=======
-      <origin xyz="0 0 0" rpy="0 1.5707 1.5707"/>
->>>>>>> master
       <mass value="5"/>
       <cylinder_inertia m="5" r="0.1" h="0.05"/>
@@ -75,9 +67,5 @@
     </visual>
     <inertial>
-<<<<<<< HEAD
       <origin rpy="0 1.5707 1.5707" xyz="0 0 0"/>
-=======
-      <origin xyz="0 0 0" rpy="0 1.5707 1.5707"/>
->>>>>>> master
       <mass value="5"/>
       <cylinder_inertia m="5" r="0.1" h="0.05"/>
@@ -141,11 +129,6 @@
       </geometry>
     </collision>
-<<<<<<< HEAD
     <visual name="visual">
       <origin rpy="0 0 3.1415" xyz="0 0 0"/>
-=======
-    <visual name="arm_back_visual">
-      <origin xyz="0 .1 0" rpy="0 1.5707 1.5707"/>
->>>>>>> master
       <geometry>
         <robot_arm />
@@ -153,9 +136,5 @@
     </visual>
     <inertial>
-<<<<<<< HEAD
       <origin xyz="0 0 0" rpy="0 0 3.1415"/>
-=======
-      <origin xyz="0 0 0" rpy="0 1.5707 1.5707"/>
->>>>>>> master
       <mass value="5"/>
       <cylinder_inertia m="5" r="0.1" h="0.05"/>
@@ -173,11 +152,6 @@
       </geometry>
     </collision>
-<<<<<<< HEAD
     <visual name="visual">
       <origin rpy="0 0 0" xyz="0 0 0"/>
-=======
-    <visual name="arm_front_visual">
-      <origin xyz="0 -.1 0" rpy="0 1.5707 1.5707"/>
->>>>>>> master
       <geometry>
         <robot_arm />
@@ -185,9 +159,5 @@
     </visual>
     <inertial>
-<<<<<<< HEAD
-      <origin xyz="0 0 0" rpy="0 0 0"/>
-=======
-      <origin xyz="0 0 0" rpy="0 1.5707 1.5707"/>
->>>>>>> master
+      <origin xyz="0 0 0" rpy="0 0 0"/>
       <mass value="5"/>
       <cylinder_inertia m="5" r="0.1" h="0.05"/>
@@ -202,9 +172,5 @@
       <origin xyz="0 0 0" rpy="0 0 1.5707"/>
       <geometry>
-<<<<<<< HEAD
         <robot_arm_drum />
-=======
-        <cylinder radius="0.1" length="0.05"/>
->>>>>>> master
       </geometry>
     </collision>
@@ -216,9 +182,5 @@
     </visual>
     <inertial>
-<<<<<<< HEAD
       <origin xyz="0 0 0" rpy="0 0 1.5707"/>
-=======
-      <origin xyz="0 0 0" rpy="0 1.5707 1.5707"/>
->>>>>>> master
       <mass value="5"/>
       <cylinder_inertia m="5" r="0.1" h="0.05"/>
@@ -233,9 +195,5 @@
       <origin xyz="0 0 0" rpy="0 0 4.7122"/>
       <geometry>
-<<<<<<< HEAD
         <robot_arm_drum />
-=======
-        <cylinder radius="0.1" length="0.05"/>
->>>>>>> master
       </geometry>
     </collision>
@@ -247,17 +205,12 @@
     </visual>
     <inertial>
-<<<<<<< HEAD
       <origin xyz="0 0 0" rpy="0 0 4.7122"/>
-=======
-      <origin xyz="0 0 0" rpy="0 1.5707 1.5707"/>
->>>>>>> master
-      <mass value="5"/>
-      <cylinder_inertia m="5" r="0.1" h="0.05"/>
-      <inertia
-        ixx="1.0" ixy="0.0" ixz="0.0"
-        iyy="1.0" iyz="0.0"
-        izz="1.0"/>
-    </inertial>
-<<<<<<< HEAD
+      <mass value="5"/>
+      <cylinder_inertia m="5" r="0.1" h="0.05"/>
+      <inertia
+        ixx="1.0" ixy="0.0" ixz="0.0"
+        iyy="1.0" iyz="0.0"
+        izz="1.0"/>
+    </inertial>
   </link>
 <!-- Transmissions -->
@@ -302,96 +255,4 @@
     </actuator>
   </transmission>
-=======
-  </link>
-  <!--First Camera Added/-->
-  <link name="f_stereo_1">
-    <collision>
-      <origin xyz="0 0 0" rpy="0 0 0"/>
-      <geometry>
-        <box size="${cameraSize} ${cameraSize} ${cameraSize}"/>
-      </geometry>
-    </collision>
-    <visual>
-      <origin xyz="0 0 0" rpy="0 0 0"/>
-      <geometry>
-        <box size="${cameraSize} ${cameraSize} ${cameraSize}"/>
-      </geometry>
-      <material name="green"/>
-    </visual>
-    <inertial>
-      <mass value="${cameraMass}" />
-      <origin xyz="0 0 0" rpy="0 0 0"/>
-      <box_inertia m="${cameraMass}" x="${cameraSize}" y="${cameraSize}" z="${cameraSize}" />
-      <inertia ixx="1e-6" ixy="0" ixz="0" iyy="1e-6" iyz="0" izz="1e-6" />
-    </inertial>
-  </link>
-  <!--Second Camera Added/-->
-  <link name="f_stereo_2">
-    <collision>
-      <origin xyz="0 0 0" rpy="0 0 0"/>
-      <geometry>
-        <box size="${cameraSize} ${cameraSize} ${cameraSize}"/>
-      </geometry>
-    </collision>
-    <visual>
-      <origin xyz="0 0 0" rpy="0 0 0"/>
-      <geometry>
-        <box size="${cameraSize} ${cameraSize} ${cameraSize}"/>
-      </geometry>
-      <material name="green"/>
-    </visual>
-    <inertial>
-      <mass value="${cameraMass}" />
-      <origin xyz="0 0 0" rpy="0 0 0"/>
-      <box_inertia m="${cameraMass}" x="${cameraSize}" y="${cameraSize}" z="${cameraSize}" />
-      <inertia ixx="1e-6" ixy="0" ixz="0" iyy="1e-6" iyz="0" izz="1e-6" />
-    </inertial>
-  </link>
-    <!--Third Camera Added/-->
-  <link name="f_stereo_3">
-    <collision>
-      <origin xyz="0 0 0" rpy="0 0 0"/>
-      <geometry>
-        <box size="${cameraSize} ${cameraSize} ${cameraSize}"/>
-      </geometry>
-    </collision>
-    <visual>
-      <origin xyz="0 0 0" rpy="0 0 0"/>
-      <geometry>
-        <box size="${cameraSize} ${cameraSize} ${cameraSize}"/>
-      </geometry>
-      <material name="green"/>
-    </visual>
-    <inertial>
-      <mass value="${cameraMass}" />
-      <origin xyz="0 0 0" rpy="0 0 0"/>
-      <box_inertia m="${cameraMass}" x="${cameraSize}" y="${cameraSize}" z="${cameraSize}" />
-      <inertia ixx="1e-6" ixy="0" ixz="0" iyy="1e-6" iyz="0" izz="1e-6" />
-    </inertial>
-  </link>
-      <!--Fourth Camera Added/-->
-  <link name="f_stereo_4">
-    <collision>
-      <origin xyz="0 0 0" rpy="0 0 0"/>
-      <geometry>
-        <box size="${cameraSize} ${cameraSize} ${cameraSize}"/>
-      </geometry>
-    </collision>
-    <visual>
-      <origin xyz="0 0 0" rpy="0 0 0"/>
-      <geometry>
-        <box size="${cameraSize} ${cameraSize} ${cameraSize}"/>
-      </geometry>
-      <material name="green"/>
-    </visual>
-    <inertial>
-      <mass value="${cameraMass}" />
-      <origin xyz="0 0 0" rpy="0 0 0"/>
-      <box_inertia m="${cameraMass}" x="${cameraSize}" y="${cameraSize}" z="${cameraSize}" />
-      <inertia ixx="1e-6" ixy="0" ixz="0" iyy="1e-6" iyz="0" izz="1e-6" />
-    </inertial>
-  </link>
-  <!--Below are all of the robot's joints/-->
->>>>>>> master
   <transmission name="arm_front_tran">
     <type>transmission_interface/SimpleTransmission</type>
@@ -489,5 +350,4 @@
   <joint name="camera_front_joint" type="fixed">
     <axis xyz="0 1 0" />
-<<<<<<< HEAD
     <origin xyz=".75 0 0" rpy="0 0 0"/>
     <parent link="base_link"/>
@@ -499,27 +359,4 @@
     <parent link="base_link"/>
     <child link="stereo_camera_back"/>
-=======
-    <origin xyz=".47 .03 0" rpy="0 0 0"/>
-    <parent link="base_link"/>
-    <child link="f_stereo_1"/>
-  </joint>
-  <joint name="camera_joint2" type="fixed">
-    <axis xyz="0 1 0" />
-    <origin xyz=".47 -.03 0" rpy="0 0 0"/>
-    <parent link="base_link"/>
-    <child link="f_stereo_2"/>
-  </joint>
-  <joint name="camera_joint3" type="fixed">
-    <axis xyz="0 1 0" />
-    <origin xyz="-.47 .03 0" rpy="0 0 3.14"/>
-    <parent link="base_link"/>
-    <child link="f_stereo_3"/>
-  </joint>
-  <joint name="camera_joint4" type="fixed">
-    <axis xyz="0 1 0" />
-    <origin xyz="-.47 -.03 0" rpy="0 0 3.14"/>
-    <parent link="base_link"/>
-    <child link="f_stereo_4"/>
->>>>>>> master
   </joint>
   <joint type="continuous" name="left_wheel_front_hinge">
@@ -556,9 +393,5 @@
   </joint>
   <joint type="continuous" name="arm_back_hinge">
-<<<<<<< HEAD
     <origin xyz="-0.25 0 0" rpy="0 0 6.2828"/>
-=======
-    <origin xyz="-0.2 0 0" rpy="0 0 1.57"/>
->>>>>>> master
     <child link="arm_back"/>
     <parent link="base_link"/>
@@ -568,9 +401,5 @@
   </joint>
   <joint type="continuous" name="arm_front_hinge">
-<<<<<<< HEAD
     <origin xyz="0.25 0 0" rpy="0 0 6.2828"/>
-=======
-    <origin xyz="0.2 0 0" rpy="0 0 1.57"/>
->>>>>>> master
     <child link="arm_front"/>
     <parent link="base_link"/>
@@ -580,9 +409,5 @@
   </joint>
   <joint type="continuous" name="drum_front_hinge">
-<<<<<<< HEAD
     <origin xyz="0.338245 0 0" rpy="0 0 6.2828"/>
-=======
-    <origin xyz="0 -0.2 0" rpy="0 0 1.57"/>
->>>>>>> master
     <child link="drum_front"/>
     <parent link="arm_front"/>
@@ -592,9 +417,5 @@
   </joint>
   <joint type="continuous" name="drum_back_hinge">
-<<<<<<< HEAD
     <origin xyz="-0.338245 0 0" rpy="0 0 6.2828"/>
-=======
-    <origin xyz="0 0.2 0" rpy="0 0 1.57"/>
->>>>>>> master
     <child link="drum_back"/>
     <parent link="arm_back"/>

Commit message: Added drum movement to sim

File: packages/ai_swarm/ez_rassor_description/urdf/ez_rassor.xacro (robot description, xacro)
@@ -275,4 +275,24 @@
     </actuator>
   </transmission>
+  <transmission name="drum_front_hinge_tran">
+    <type>transmission_interface/SimpleTransmission</type>
+    <joint name="drum_front_hinge">
+      <hardwareInterface>hardware_interface/VelocityJointInterface</hardwareInterface>
+    </joint>
+    <actuator name="drum_front_hinge_motor">
+      <hardwareInterface>hardware_interface/VelocityJointInterface</hardwareInterface>
+      <mechanicalReduction>1</mechanicalReduction>
+    </actuator>
+  </transmission>
+  <transmission name="drum_back_hinge_tran">
+    <type>transmission_interface/SimpleTransmission</type>
+    <joint name="drum_back_hinge">
+      <hardwareInterface>hardware_interface/VelocityJointInterface</hardwareInterface>
+    </joint>
+    <actuator name="drum_back_hinge_motor">
+      <hardwareInterface>hardware_interface/VelocityJointInterface</hardwareInterface>
+      <mechanicalReduction>1</mechanicalReduction>
+    </actuator>
+  </transmission>
   <!--Front Camera Added/-->
   <link name="stereo_camera_front">
