Commit message: New drum models added to sim

File: packages/ez_rassor/ez_rassor_description/urdf/macros.xacro (robot description, xacro)
@@ -23,5 +23,5 @@
     </macro>
     <macro name="robot_arm_drum">
-        <mesh filename="package://ez_rassor_description/meshes/drum.dae" scale="1.5 1.5 1.5"></mesh>
+        <mesh filename="package://ez_rassor_description/meshes/drum.dae" scale="0.065 0.08 0.08"></mesh>
     </macro>
     <macro name="robot_wheel">
