Commit message: Redesign of the EZ-RASSOR to create a V2 modeled after the RASSOR

File: packages/simulation/ez_rassor_description/urdf/v1_model/ez_rassor.xacro (robot description, xacro)
@@ -1,5 +1,5 @@
 <?xml version='1.0'?>
 <robot name="ez_rassor" xmlns:xacro="http://www.ros.org/wiki/xacro">
-  <xacro:property name="cameraSize" value="0.05"/>
+  <xacro:property name="cameraSize" value="0.005"/>
   <xacro:property name="cameraMass" value="0.1"/>
   <xacro:include filename="$(find ez_rassor_description)/urdf/ez_rassor.gazebo" />
@@ -8,8 +8,8 @@
   <!--Below are all of the robot's Links/-->
   <link name='base_link'>
-    <pose>0 0 0 0 0 0</pose>
+    <pose>0 0 0.1 0 0 0</pose>
     <inertial>
       <mass value="10.0"/>
-      <origin xyz="0 0 0" rpy=" 0 0 0"/>
+      <origin xyz="0.0 0 0.1" rpy=" 0 0 0"/>
       <inertia
           ixx="0.5" ixy="0" ixz="0"
@@ -19,7 +19,6 @@
     </inertial>
     <collision name='collision'>
-      <origin xyz="0 0 0" rpy=" 0 0 0"/>
-      <geometry>
-        <base_unit/>
+      <geometry>
+        <box size=".4 .2 .1"/>
       </geometry>
     </collision>
@@ -27,5 +26,5 @@
       <origin xyz="0 0 0" rpy=" 0 0 0"/>
       <geometry>
-        <base_unit/>
+        <box size=".4 .2 .1"/>
       </geometry>
     </visual>
@@ -33,5 +32,5 @@
   <link name="left_wheel_front">
     <collision name="collision">
-      <origin xyz="0 0 0" rpy="0 0 0"/>
+      <origin xyz="0 -0.06 0" rpy="3.14159 1.57079 -1.57089"/>
       <geometry>
         <robot_wheel />
@@ -39,11 +38,11 @@
     </collision>
     <visual name="left_wheel_front_visual">
-      <origin xyz="0 0 0" rpy="0 0 0"/>
-      <geometry>
-        <robot_wheel />
-      </geometry>
-    </visual>
-    <inertial>
-      <origin xyz="0 0 0" rpy="0 0 0" />
+      <origin xyz="0 -0.06 0" rpy="-3.12268 1.57079 -1.55198"/>
+      <geometry>
+        <robot_wheel />
+      </geometry>
+    </visual>
+    <inertial>
+      <origin xyz="0 0 0" rpy="0 1.5707 1.5707" />
       <mass value="5"/>
       <cylinder_inertia m="5" r="0.1" h="0.05"/>
@@ -56,5 +55,5 @@
   <link name="right_wheel_front">
     <collision name="collision">
-      <origin xyz="0 0 0" rpy="0 0 3.14159"/>
+      <origin xyz="0 0.06 0" rpy="0 1.57079 -1.57089"/>
       <geometry>
         <robot_wheel />
@@ -62,11 +61,11 @@
     </collision>
     <visual name="right_wheel_front_visual">
-      <origin xyz="0 0 0" rpy="0 0 3.14159"/>
-      <geometry>
-        <robot_wheel />
-      </geometry>
-    </visual>
-    <inertial>
-      <origin xyz="0 0 0" rpy="0 0 3.14159"/>
+      <origin xyz="0 0.06 0" rpy="-0.00702 1.57079 -1.57316"/>
+      <geometry>
+        <robot_wheel />
+      </geometry>
+    </visual>
+    <inertial>
+      <origin rpy="0 1.5707 1.5707" xyz="0 0 0"/>
       <mass value="5"/>
       <cylinder_inertia m="5" r="0.1" h="0.05"/>
@@ -79,5 +78,5 @@
   <link name="left_wheel_back">
     <collision name="collision">
-      <origin xyz="0 0 0" rpy="0 0 0"/>
+      <origin xyz="0 -0.06 0" rpy="3.14159  1.57079 -1.57089"/>
       <geometry>
         <robot_wheel />
@@ -85,11 +84,11 @@
     </collision>
     <visual name="left_wheel_back_visual">
-      <origin xyz="0 0 0" rpy="0 0 0"/>
-      <geometry>
-        <robot_wheel />
-      </geometry>
-    </visual>
-    <inertial>
-      <origin xyz="0 0 0" rpy="0 0 0"/>
+      <origin xyz="0 -0.06 0" rpy="-3.12268  1.57079 -1.55198"/>
+      <geometry>
+        <robot_wheel />
+      </geometry>
+    </visual>
+    <inertial>
+      <origin xyz="0 0 0" rpy="0 1.5707 1.5707"/>
       <mass value="5"/>
       <cylinder_inertia m="5" r="0.1" h="0.05"/>
@@ -102,5 +101,5 @@
   <link name="right_wheel_back">
     <collision name="collision">
-      <origin xyz="0 0 0" rpy="0 0 3.14159"/>
+      <origin xyz="0 0.06 0" rpy="0 1.57079 -1.57089"/>
       <geometry>
         <robot_wheel />
@@ -108,11 +107,34 @@
     </collision>
     <visual name="right_wheel_back_visual">
-      <origin xyz="0 0 0" rpy="0 0 3.14159"/>
-      <geometry>
-        <robot_wheel />
-      </geometry>
-    </visual>
-    <inertial>
-      <origin xyz="0 0 0" rpy="0 0 3.14159"/>
+      <origin xyz="0 0.06 0" rpy="-0.00702 1.57079 -1.57316"/>
+      <geometry>
+        <robot_wheel />
+      </geometry>
+    </visual>
+    <inertial>
+      <origin xyz="0 0 0" rpy="0 1.5707 1.5707"/>
+      <mass value="5"/>
+      <cylinder_inertia m="5" r="0.1" h="0.05"/>
+      <inertia
+        ixx="1.0" ixy="0.0" ixz="0.0"
+        iyy="1.0" iyz="0.0"
+        izz="1.0"/>
+    </inertial>
+  </link>
+  <link name="arm_back">
+    <collision name="collision">
+      <origin rpy="0 0 3.1415" xyz="0 0 0"/>
+      <geometry>
+        <robot_arm />
+      </geometry>
+    </collision>
+    <visual name="visual">
+      <origin rpy="0 0 3.1415" xyz="0 0 0"/>
+      <geometry>
+        <robot_arm />
+      </geometry>
+    </visual>
+    <inertial>
+      <origin xyz="0 0 0" rpy="0 0 3.1415"/>
       <mass value="5"/>
       <cylinder_inertia m="5" r="0.1" h="0.05"/>
@@ -125,40 +147,17 @@
   <link name="arm_front">
     <collision name="collision">
-      <origin xyz="0 0 0" rpy="0 0 0"/>
-      <geometry>
-        <drum_arm />
+      <origin rpy="0 0 0" xyz="0 0 0"/>
+      <geometry>
+        <robot_arm />
       </geometry>
     </collision>
     <visual name="visual">
-      <origin xyz="0 0 0" rpy="0 0 0" />
-      <geometry>
-        <drum_arm />
-      </geometry>
-    </visual>
-    <inertial>
-      <origin xyz="0 0 0" rpy="0 0 0"/>
-      <mass value="5"/>
-      <cylinder_inertia m="5" r="0.1" h="0.05"/>
-      <inertia
-        ixx="1.0" ixy="0.0" ixz="0.0"
-        iyy="1.0" iyz="0.0"
-        izz="1.0"/>
-    </inertial>
-  </link>
-  <link name="arm_back">
-    <collision name="collision">
-      <origin xyz="0 0 0" rpy="0 0 3.1415"/>
-      <geometry>
-        <drum_arm />
-      </geometry>
-    </collision>
-    <visual name="visual">
-      <origin xyz="0 0 0" rpy="0 0 3.1415"/>
-      <geometry>
-        <drum_arm />
-      </geometry>
-    </visual>
-    <inertial>
-      <origin xyz="0 0 0" rpy="0 0 3.1415"/>
+      <origin rpy="0 0 0" xyz="0 0 0"/>
+      <geometry>
+        <robot_arm />
+      </geometry>
+    </visual>
+    <inertial>
+      <origin xyz="0 0 0" rpy="0 0 0"/>
       <mass value="5"/>
       <cylinder_inertia m="5" r="0.1" h="0.05"/>
@@ -171,5 +170,5 @@
   <link name="drum_front">
     <collision name="collision">
-      <origin xyz="0 0 0" rpy="0 0 0"/>
+      <origin xyz="0 0 0" rpy="0 0 1.5707"/>
       <geometry>
         <robot_arm_drum />
@@ -177,5 +176,5 @@
     </collision>
     <visual name="drum_front_visual">
-      <origin xyz="0 0 0" rpy="0 0 0"/>
+      <origin xyz="0 0 0" rpy="0 0 1.5707"/>
       <geometry>
         <robot_arm_drum />
@@ -183,5 +182,5 @@
     </visual>
     <inertial>
-      <origin xyz="0 0 0" rpy="0 0 0"/>
+      <origin xyz="0 0 0" rpy="0 0 1.5707"/>
       <mass value="5"/>
       <cylinder_inertia m="5" r="0.1" h="0.05"/>
@@ -194,5 +193,5 @@
   <link name="drum_back">
     <collision name="collision">
-      <origin xyz="0 0 0" rpy="0 0 3.14159"/>
+      <origin xyz="0 0 0" rpy="0 0 4.7122"/>
       <geometry>
         <robot_arm_drum />
@@ -200,5 +199,5 @@
     </collision>
     <visual name="drum_back">
-      <origin xyz="0 0 0" rpy="0 0 3.14159"/>
+      <origin xyz="0 0 0" rpy="0 0 4.7122"/>
       <geometry>
         <robot_arm_drum />
@@ -206,14 +205,24 @@
     </visual>
     <inertial>
-      <origin xyz="0 0 0" rpy="0 0 3.14159"/>
-      <mass value="5"/>
-      <cylinder_inertia m="5" r="0.1" h="0.05"/>
-      <inertia
-        ixx="1.0" ixy="0.0" ixz="0.0"
-        iyy="1.0" iyz="0.0"
-        izz="1.0"/>
-    </inertial>
-  </link>
-  <!-- Transmissions -->
+      <origin xyz="0 0 0" rpy="0 0 4.7122"/>
+      <mass value="5"/>
+      <cylinder_inertia m="5" r="0.1" h="0.05"/>
+      <inertia
+        ixx="1.0" ixy="0.0" ixz="0.0"
+        iyy="1.0" iyz="0.0"
+        izz="1.0"/>
+    </inertial>
+  </link>
+<!-- Transmissions -->
+<transmission name="left_wheel_back_tran">
+    <type>transmission_interface/SimpleTransmission</type>
+    <joint name="left_wheel_back_hinge">
+      <hardwareInterface>hardware_interface/VelocityJointInterface</hardwareInterface>
+    </joint>
+    <actuator name="left_wheel_back_motor">
+      <hardwareInterface>hardware_interface/VelocityJointInterface</hardwareInterface>
+      <mechanicalReduction>1</mechanicalReduction>
+    </actuator>
+  </transmission>
   <transmission name="left_wheel_front_tran">
     <type>transmission_interface/SimpleTransmission</type>
@@ -226,10 +235,10 @@
     </actuator>
   </transmission>
-  <transmission name="left_wheel_back_tran">
-    <type>transmission_interface/SimpleTransmission</type>
-    <joint name="left_wheel_back_hinge">
-      <hardwareInterface>hardware_interface/VelocityJointInterface</hardwareInterface>
-    </joint>
-    <actuator name="left_wheel_back_motor">
+  <transmission name="right_wheel_back_tran">
+    <type>transmission_interface/SimpleTransmission</type>
+    <joint name="right_wheel_back_hinge">
+      <hardwareInterface>hardware_interface/VelocityJointInterface</hardwareInterface>
+    </joint>
+    <actuator name="right_wheel_back_motor">
       <hardwareInterface>hardware_interface/VelocityJointInterface</hardwareInterface>
       <mechanicalReduction>1</mechanicalReduction>
@@ -246,14 +255,4 @@
     </actuator>
   </transmission>
-  <transmission name="right_wheel_back_tran">
-    <type>transmission_interface/SimpleTransmission</type>
-    <joint name="right_wheel_back_hinge">
-      <hardwareInterface>hardware_interface/VelocityJointInterface</hardwareInterface>
-    </joint>
-    <actuator name="right_wheel_back_motor">
-      <hardwareInterface>hardware_interface/VelocityJointInterface</hardwareInterface>
-      <mechanicalReduction>1</mechanicalReduction>
-    </actuator>
-  </transmission>
   <transmission name="arm_front_tran">
     <type>transmission_interface/SimpleTransmission</type>
@@ -296,5 +295,5 @@
     </actuator>
   </transmission>
-  <!-- Front Camera Added -->
+  <!--Front Camera Added/-->
   <link name="stereo_camera_front">
     <collision>
@@ -318,4 +317,5 @@
     </inertial>
   </link>
+<!--Back Camera Added/-->
   <link name="stereo_camera_back">
     <collision>
@@ -339,4 +339,5 @@
     </inertial>
   </link>
+    <!-- IMU -->
   <link name="imu_link">
     <collision>
@@ -366,18 +367,19 @@
     <child link="imu_link"/>
   </joint>
+  <!--Below are all of the robot's joints/-->
   <joint name="camera_front_joint" type="fixed">
-    <origin xyz=".75 0 0" rpy="0 0.785 0"/>
     <axis xyz="0 1 0" />
+    <origin xyz=".75 0 0" rpy="0 0 0"/>
     <parent link="base_link"/>
     <child link="stereo_camera_front"/>
   </joint>
   <joint name="camera_back_joint" type="fixed">
-    <origin xyz="-.5 0.005 0" rpy="0 -0.785 3.14"/>
     <axis xyz="0 1 0" />
-    <parent link="arm_back" />
+    <origin xyz="-.75 0 0" rpy="0 0 3.14"/>
+    <parent link="base_link"/>
     <child link="stereo_camera_back"/>
   </joint>
   <joint type="continuous" name="left_wheel_front_hinge">
-    <origin xyz="0.20 0.285 0" rpy="0 0 0"/>
+    <origin xyz="0.15 0.15 0" rpy="0 0 0"/>
     <child link="left_wheel_front"/>
     <parent link="base_link"/>
@@ -387,5 +389,5 @@
   </joint>
   <joint type="continuous" name="right_wheel_front_hinge">
-    <origin xyz="0.20 -0.285 0" rpy="0 0 0"/>
+    <origin xyz="0.15 -0.15 0" rpy="0 0 0"/>
     <child link="right_wheel_front"/>
     <parent link="base_link"/>
@@ -395,5 +397,5 @@
   </joint>
   <joint type="continuous" name="left_wheel_back_hinge">
-    <origin xyz="-0.20 0.285 0" rpy="0 0 0"/>
+    <origin xyz="-0.15 0.15 0" rpy="0 0 0"/>
     <child link="left_wheel_back"/>
     <parent link="base_link"/>
@@ -403,5 +405,5 @@
   </joint>
   <joint type="continuous" name="right_wheel_back_hinge">
-    <origin xyz="-0.20 -0.285 0" rpy="0 0 0"/>
+    <origin xyz="-0.15 -0.15 0" rpy="0 0 0"/>
     <child link="right_wheel_back"/>
     <parent link="base_link"/>
@@ -410,6 +412,14 @@
     <joint_properties damping="0.0" friction="0.0"/>
   </joint>
+  <joint type="continuous" name="arm_back_hinge">
+    <origin xyz="-0.25 0 0" rpy="0 0 6.2828"/>
+    <child link="arm_back"/>
+    <parent link="base_link"/>
+    <axis xyz="0 1 0" rpy="0 0 0"/>
+    <limit effort="100" velocity="100"/>
+    <joint_properties damping="0.0" friction="0.0"/>
+  </joint>
   <joint type="continuous" name="arm_front_hinge">
-    <origin xyz="0.20 0 0" rpy="0 0 0"/>
+    <origin xyz="0.25 0 0" rpy="0 0 6.2828"/>
     <child link="arm_front"/>
     <parent link="base_link"/>
@@ -418,14 +428,6 @@
     <joint_properties damping="0.0" friction="0.0"/>
   </joint>
-  <joint type="continuous" name="arm_back_hinge">
-    <origin xyz="-0.20 0 0" rpy="0 0 0"/>
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
File: packages/simulation/ez_rassor_description/urdf/v1_model/macros.xacro (robot description, xacro)
@@ -23,14 +23,8 @@
     </macro>
     <macro name="robot_arm_drum">
-        <mesh filename="package://ez_rassor_description/meshes/drum.dae" scale="0.35 0.35 0.35"></mesh>
+        <mesh filename="package://ez_rassor_description/meshes/drum.dae" scale=".07 .09 .09"></mesh>
     </macro>
     <macro name="robot_wheel">
-        <mesh filename="package://ez_rassor_description/meshes/wheel.dae" scale="0.35 0.35 0.35"></mesh>
-    </macro>
-    <macro name="base_unit">
-        <mesh filename="package://ez_rassor_description/meshes/base_unit.dae" scale="0.35 0.35 0.35"></mesh>
-    </macro>
-    <macro name="drum_arm">
-        <mesh filename="package://ez_rassor_description/meshes/drum_arm.dae" scale="0.35 0.35 0.35"></mesh>
+        <mesh filename="package://ez_rassor_description/meshes/wheel.dae" scale="1.2 1.2 1.2"></mesh>
     </macro>
 </robot>
