Commit message: storing my changes

File: packages/simulation/ez_rassor_description/urdf/macros.xacro (robot description, xacro)
@@ -23,8 +23,8 @@
     </macro>
     <macro name="robot_arm_drum">
-        <mesh filename="package://ez_rassor_description/meshes/drum.dae" scale="0.065 0.08 0.08"></mesh>
+        <mesh filename="package://ez_rassor_description/meshes/drum.dae" scale=".09 .13 .13"></mesh>
     </macro>
     <macro name="robot_wheel">
-        <mesh filename="package://ez_rassor_description/meshes/wheel.dae" scale="1.1 1.1 1.1"></mesh>
+        <mesh filename="package://ez_rassor_description/meshes/wheel.dae" scale="1.2 1.2 1.2"></mesh>
     </macro>
 </robot>

Commit message: Object Avoidance Fully Completed

File: packages/simulation/ez_rassor_description/urdf/macros.xacro (robot description, xacro)
@@ -23,5 +23,5 @@
     </macro>
     <macro name="robot_arm_drum">
-        <mesh filename="package://ez_rassor_description/meshes/drum.dae" scale=".09 .13 .13"></mesh>
+        <mesh filename="package://ez_rassor_description/meshes/drum.dae" scale=".07 .09 .09"></mesh>
     </macro>
     <macro name="robot_wheel">

Commit message: Adds a forcetorque sensor to the gazebo references

File: packages/simulation/ez_rassor_description/urdf/macros.xacro (robot description, xacro)
@@ -1,4 +1,5 @@
 <?xml version='1.0'?>
 <robot name="ez_rassor" xmlns:xacro="http://www.ros.org/wiki/xacro">
+    <!-- Inertia Tensors Used: https://en.wikipedia.org/wiki/List_of_moments_of_inertia#List_of_3D_inertia_tensors -->
     <macro name="cylinder_inertia" params="m r h">
     <inertia  ixx="${m*(3*r*r+h*h)/12}" ixy = "0" ixz = "0"
@@ -19,4 +20,18 @@
     />
     </macro>
+    <macro name="slender_rod_along_y_inertia" params="m l mass_about">
+        <if value="${mass_about == 'end'}">
+            <inertia
+                ixx="${1/3*m*(l*l)}" ixy = "0"
+                ixz = "0" iyy="0"
+                iyz = "0" izz="${1/3*m*(l*l)}" />
+        </if>
+        <unless value="${mass_about == 'center'}">
+            <inertia
+                ixx="${1/12*m*(l*l)}" ixy = "0"
+                ixz = "0" iyy="0"
+                iyz = "0" izz="${1/12*m*(l*l)}" />
+        </unless>
+    </macro>
     <macro name="robot_arm">
         <mesh filename="package://ez_rassor_description/meshes/drum_arm_short.dae" scale="1.0 1.0 1.0"></mesh>
