Commit message: Corrects the placement of the cameras on the model.

File: packages/simulation/ez_rassor_description/urdf/ez_rassor.xacro (robot description, xacro)
@@ -367,7 +367,7 @@
   </joint>
   <joint name="camera_front_joint" type="fixed">
-    <origin xyz=".75 0 0" rpy="0 0.785 0"/>
+    <origin xyz=".5 -0.005 0" rpy="0 0.785 0"/>
     <axis xyz="0 1 0" />
-    <parent link="base_link"/>
+    <parent link="arm_front"/>
     <child link="stereo_camera_front"/>
   </joint>

Commit message: Fixed joy, ai control, and made the movement work again

File: packages/simulation/ez_rassor_description/urdf/ez_rassor.xacro (robot description, xacro)
@@ -10,5 +10,5 @@
     <pose>0 0 0 0 0 0</pose>
     <inertial>
-      <mass value="10.0"/>
+      <mass value="35.0"/>
       <origin xyz="0 0 0" rpy=" 0 0 0"/>
       <inertia

Commit message: Adding collision detection to EZ-RASSOR

File: packages/simulation/ez_rassor_description/urdf/ez_rassor.xacro (robot description, xacro)
@@ -170,9 +170,15 @@
   </link>
   <link name="drum_front">
-    <collision name="collision">
+    <!-- <collision name="collision">
       <origin xyz="0 0 0" rpy="0 0 0"/>
       <geometry>
         <robot_arm_drum />
       </geometry>
+    </collision>-->
+    <collision name="collision">
+      <origin xyz="0 0 0" rpy="0 1.5707 1.5707"/>
+      <geometry>
+        <cylinder radius="0.1839" length="1.0"/>
+      </geometry>
     </collision>
     <visual name="drum_front_visual">
@@ -193,8 +199,14 @@
   </link>
   <link name="drum_back">
-    <collision name="collision">
+    <!-- <collision name="collision">
       <origin xyz="0 0 0" rpy="0 0 3.14159"/>
       <geometry>
         <robot_arm_drum />
+      </geometry>
+    </collision> -->
+     <collision name="collision">
+      <origin xyz="0 0 0" rpy="0 1.5707 1.5707"/>
+      <geometry>
+        <cylinder radius="0.1839" length="1.0"/>
       </geometry>
     </collision>

Commit message: I'm not even sure what I changed since this was before spring break but this works.

File: packages/simulation/ez_rassor_description/urdf/ez_rassor.xacro (robot description, xacro)
@@ -367,7 +367,7 @@
   </joint>
   <joint name="camera_front_joint" type="fixed">
-    <origin xyz=".75 0 0" rpy="0 0.785 0"/>
+    <origin xyz=".5 0.005 0" rpy="0 0.785 0"/>
     <axis xyz="0 1 0" />
-    <parent link="base_link"/>
+    <parent link="arm_front"/>
     <child link="stereo_camera_front"/>
   </joint>

Commit message: Point Cloud generated.

File: packages/simulation/ez_rassor_description/urdf/ez_rassor.xacro (robot description, xacro)
@@ -367,6 +367,7 @@
   </joint>
   <joint name="camera_front_joint" type="fixed">
-    <origin xyz=".75 0 0" rpy="0 0.785 0"/>
-    <axis xyz="0 1 0" />
+    <!-- <origin xyz=".75 0 0" rpy="0 0.785 0"/> -->
+    <origin xyz="1 0 0" rpy="0 0 0"/>
+    <axis xyz="0 0 0" />
     <parent link="base_link"/>
     <child link="stereo_camera_front"/>

Commit message: Fixing inertia on EZ_RASSOR and comms fixes

File: packages/simulation/ez_rassor_description/urdf/ez_rassor.xacro (robot description, xacro)
@@ -47,5 +47,100 @@
       <origin xyz="0 0 0" rpy="0 0 0" />
       <mass value="5"/>
-      <cylinder_inertia m="5" r="0.1" h="0.05"/>
+      <cylinder_inertia m="5" r="0.18" h="0.2"/>
+    </inertial>
+  </link>
+  <link name="right_wheel_front">
+    <collision name="collision">
+      <origin xyz="0 0 0" rpy="0 0 3.14159"/>
+      <geometry>
+        <robot_wheel />
+      </geometry>
+    </collision>
+    <visual name="right_wheel_front_visual">
+      <origin xyz="0 0 0" rpy="0 0 3.14159"/>
+      <geometry>
+        <robot_wheel />
+      </geometry>
+    </visual>
+    <inertial>
+      <origin xyz="0 0 0" rpy="0 0 3.14159"/>
+      <mass value="5"/>
+      <cylinder_inertia m="5" r="0.18" h="0.2"/>
+    </inertial>
+  </link>
+  <link name="left_wheel_back">
+    <collision name="collision">
+      <origin xyz="0 0 0" rpy="0 0 0"/>
+      <geometry>
+        <robot_wheel />
+      </geometry>
+    </collision>
+    <visual name="left_wheel_back_visual">
+      <origin xyz="0 0 0" rpy="0 0 0"/>
+      <geometry>
+        <robot_wheel />
+      </geometry>
+    </visual>
+    <inertial>
+      <origin xyz="0 0 0" rpy="0 0 0"/>
+      <mass value="5"/>
+      <cylinder_inertia m="5" r="0.18" h="0.2"/>
+    </inertial>
+  </link>
+  <link name="right_wheel_back">
+    <collision name="collision">
+      <origin xyz="0 0 0" rpy="0 0 3.14159"/>
+      <geometry>
+        <robot_wheel />
+      </geometry>
+    </collision>
+    <visual name="right_wheel_back_visual">
+      <origin xyz="0 0 0" rpy="0 0 3.14159"/>
+      <geometry>
+        <robot_wheel />
+      </geometry>
+    </visual>
+    <inertial>
+      <origin xyz="0 0 0" rpy="0 0 3.14159"/>
+      <mass value="5"/>
+      <cylinder_inertia m="5" r="0.18" h="0.2"/>
+    </inertial>
+  </link>
+  <link name="arm_front">
+    <collision name="collision">
+      <origin xyz="0 0 0" rpy="0 0 0"/>
+      <geometry>
+        <drum_arm />
+      </geometry>
+    </collision>
+    <visual name="visual">
+      <origin xyz="0 0 0" rpy="0 0 0" />
+      <geometry>
+        <drum_arm />
+      </geometry>
+    </visual>
+    <inertial>
+      <origin xyz="0 0 0" rpy="0 0 0"/>
+      <mass value="5"/>
+      <cylinder_inertia m="5" r="0.05" h="0.3"/>
+    </inertial>
+  </link>
+  <link name="arm_back">
+    <collision name="collision">
+      <origin xyz="0 0 0" rpy="0 0 3.1415"/>
+      <geometry>
+        <drum_arm />
+      </geometry>
+    </collision>
+    <visual name="visual">
+      <origin xyz="0 0 0" rpy="0 0 3.1415"/>
+      <geometry>
+        <drum_arm />
+      </geometry>
+    </visual>
+    <inertial>
+      <origin xyz="0 0 0" rpy="0 0 3.1415"/>
+      <mass value="5"/>
+      <cylinder_inertia m="5" r="0.05" h="0.3"/>
       <inertia
         ixx="1.0" ixy="0.0" ixz="0.0"
@@ -54,119 +149,4 @@
     </inertial>
   </link>
-  <link name="right_wheel_front">
-    <collision name="collision">
-      <origin xyz="0 0 0" rpy="0 0 3.14159"/>
-      <geometry>
-        <robot_wheel />
-      </geometry>
-    </collision>
-    <visual name="right_wheel_front_visual">
-      <origin xyz="0 0 0" rpy="0 0 3.14159"/>
-      <geometry>
-        <robot_wheel />
-      </geometry>
-    </visual>
-    <inertial>
-      <origin xyz="0 0 0" rpy="0 0 3.14159"/>
-      <mass value="5"/>
-      <cylinder_inertia m="5" r="0.1" h="0.05"/>
-      <inertia
-        ixx="1.0" ixy="0.0" ixz="0.0"
-        iyy="1.0" iyz="0.0"
-        izz="1.0"/>
-    </inertial>
-  </link>
-  <link name="left_wheel_back">
-    <collision name="collision">
-      <origin xyz="0 0 0" rpy="0 0 0"/>
-      <geometry>
-        <robot_wheel />
-      </geometry>
-    </collision>
-    <visual name="left_wheel_back_visual">
-      <origin xyz="0 0 0" rpy="0 0 0"/>
-      <geometry>
-        <robot_wheel />
-      </geometry>
-    </visual>
-    <inertial>
-      <origin xyz="0 0 0" rpy="0 0 0"/>
-      <mass value="5"/>
-      <cylinder_inertia m="5" r="0.1" h="0.05"/>
-      <inertia
-        ixx="1.0" ixy="0.0" ixz="0.0"
-        iyy="1.0" iyz="0.0"
-        izz="1.0"/>
-    </inertial>
-  </link>
-  <link name="right_wheel_back">
-    <collision name="collision">
-      <origin xyz="0 0 0" rpy="0 0 3.14159"/>
-      <geometry>
-        <robot_wheel />
-      </geometry>
-    </collision>
-    <visual name="right_wheel_back_visual">
-      <origin xyz="0 0 0" rpy="0 0 3.14159"/>
-      <geometry>
-        <robot_wheel />
-      </geometry>
-    </visual>
-    <inertial>
-      <origin xyz="0 0 0" rpy="0 0 3.14159"/>
-      <mass value="5"/>
-      <cylinder_inertia m="5" r="0.1" h="0.05"/>
-      <inertia
-        ixx="1.0" ixy="0.0" ixz="0.0"
-        iyy="1.0" iyz="0.0"
-        izz="1.0"/>
-    </inertial>
-  </link>
-  <link name="arm_front">
-    <collision name="collision">
-      <origin xyz="0 0 0" rpy="0 0 0"/>
-      <geometry>
-        <drum_arm />
-      </geometry>
-    </collision>
-    <visual name="visual">
-      <origin xyz="0 0 0" rpy="0 0 0" />
-      <geometry>
-        <drum_arm />
-      </geometry>
-    </visual>
-    <inertial>
-      <origin xyz="0 0 0" rpy="0 0 0"/>
-      <mass value="5"/>
-      <cylinder_inertia m="5" r="0.1" h="0.05"/>
-      <inertia
-        ixx="1.0" ixy="0.0" ixz="0.0"
-        iyy="1.0" iyz="0.0"
-        izz="1.0"/>
-    </inertial>
-  </link>
-  <link name="arm_back">
-    <collision name="collision">
-      <origin xyz="0 0 0" rpy="0 0 3.1415"/>
-      <geometry>
-        <drum_arm />
-      </geometry>
-    </collision>
-    <visual name="visual">
-      <origin xyz="0 0 0" rpy="0 0 3.1415"/>
-      <geometry>
-        <drum_arm />
-      </geometry>
-    </visual>
-    <inertial>
-      <origin xyz="0 0 0" rpy="0 0 3.1415"/>
-      <mass value="5"/>
-      <cylinder_inertia m="5" r="0.1" h="0.05"/>
-      <inertia
-        ixx="1.0" ixy="0.0" ixz="0.0"
-        iyy="1.0" iyz="0.0"
-        izz="1.0"/>
-    </inertial>
-  </link>
   <link name="drum_front">
     <!-- <collision name="collision">
@@ -191,9 +171,5 @@
       <origin xyz="0 0 0" rpy="0 0 0"/>
       <mass value="5"/>
-      <cylinder_inertia m="5" r="0.1" h="0.05"/>
-      <inertia
-        ixx="1.0" ixy="0.0" ixz="0.0"
-        iyy="1.0" iyz="0.0"
-        izz="1.0"/>
+      <cylinder_inertia m="5" r="0.1839" h="1.0"/>
     </inertial>
   </link>
@@ -220,9 +196,5 @@
       <origin xyz="0 0 0" rpy="0 0 3.14159"/>
       <mass value="5"/>
-      <cylinder_inertia m="5" r="0.1" h="0.05"/>
-      <inertia
-        ixx="1.0" ixy="0.0" ixz="0.0"
-        iyy="1.0" iyz="0.0"
-        izz="1.0"/>
+      <cylinder_inertia m="5" r="0.1839" h="1.0"/>
     </inertial>
   </link>

File: packages/simulation/ez_rassor_description/urdf/macros.xacro (robot description, xacro)
@@ -3,7 +3,8 @@
     <!-- Inertia Tensors Used: https://en.wikipedia.org/wiki/List_of_moments_of_inertia#List_of_3D_inertia_tensors -->
     <macro name="cylinder_inertia" params="m r h">
-    <inertia  ixx="${m*(3*r*r+h*h)/12}" ixy = "0" ixz = "0"
-        iyy="${m*(3*r*r+h*h)/12}" iyz = "0"
-        izz="${m*r*r/2}"
+    <inertia
+        ixx="${m*((3*r*r)+(h*h))/12}" ixy = "0"                 ixz = "0"
+                                  iyy="${m*((3*r*r)+(h*h))/12}" iyz = "0"
+                                                            izz="${(m*(r*r))/2}"
     />
     </macro>
@@ -34,4 +35,5 @@
         </unless>
     </macro>
+    <!-- VISUAL AND COLLISION MACROS -->
     <macro name="robot_arm">
         <mesh filename="package://ez_rassor_description/meshes/drum_arm_short.dae" scale="1.0 1.0 1.0"></mesh>

Commit message: Semi Working Navigation

File: packages/simulation/ez_rassor_description/urdf/ez_rassor.xacro (robot description, xacro)
@@ -169,11 +169,11 @@
     </inertial>
   </link>
-  <link name="drum_front">
-    <!-- <collision name="collision">
+ <link name="drum_front">
+    <collision name="collision">
       <origin xyz="0 0 0" rpy="0 0 0"/>
       <geometry>
         <robot_arm_drum />
       </geometry>
-    </collision>-->
+    </collision>
     <collision name="collision">
       <origin xyz="0 0 0" rpy="0 1.5707 1.5707"/>
@@ -190,6 +190,6 @@
     <inertial>
       <origin xyz="0 0 0" rpy="0 0 0"/>
-      <mass value="5"/>
-      <cylinder_inertia m="5" r="0.1" h="0.05"/>
+      <mass value=".5"/>
+      <cylinder_inertia m=".5" r="0.1" h="0.05"/>
       <inertia
         ixx="1.0" ixy="0.0" ixz="0.0"
@@ -199,10 +199,10 @@
   </link>
   <link name="drum_back">
-    <!-- <collision name="collision">
+    <collision name="collision">
       <origin xyz="0 0 0" rpy="0 0 3.14159"/>
       <geometry>
         <robot_arm_drum />
       </geometry>
-    </collision> -->
+    </collision>
      <collision name="collision">
       <origin xyz="0 0 0" rpy="0 1.5707 1.5707"/>
@@ -219,6 +219,6 @@
     <inertial>
       <origin xyz="0 0 0" rpy="0 0 3.14159"/>
-      <mass value="5"/>
-      <cylinder_inertia m="5" r="0.1" h="0.05"/>
+      <mass value=".5"/>
+      <cylinder_inertia m=".5" r="0.1" h="0.05"/>
       <inertia
         ixx="1.0" ixy="0.0" ixz="0.0"

Commit message: Computer is broken - saving work

File: packages/simulation/ez_rassor_description/urdf/ez_rassor.xacro (robot description, xacro)
@@ -302,25 +302,5 @@
     </inertial>
   </link>
-  <link name="stereo_camera_back">
-    <collision>
-      <origin xyz="0 0 0" rpy="0 0 0"/>
-      <geometry>
-        <box size="${cameraSize} ${cameraSize} ${cameraSize}"/>
-      </geometry>
-    </collision>
-    <visual>
-      <origin xyz="0 0 0" rpy="0 0 0"/>
-      <geometry>
-        <box size="${cameraSize} ${cameraSize} ${cameraSize}"/>
-      </geometry>
-      <material name="green"/>
-    </visual>
-    <inertial>
-      <mass value="${cameraMass}" />
-      <origin xyz="0 0 0" rpy="0 0 0"/>
-      <box_inertia m="${cameraMass}" x="${cameraSize}" y="${cameraSize}" z="${cameraSize}" />
-      <inertia ixx="1e-6" ixy="0" ixz="0" iyy="1e-6" iyz="0" izz="1e-6" />
-    </inertial>
-  </link>
+  <!-- IMU -->
   <link name="imu_link">
     <collision>
@@ -351,14 +331,8 @@
   </joint>
   <joint name="camera_front_joint" type="fixed">
-    <origin xyz=".5 -0.005 0" rpy="0 0.785 0"/>
+    <origin xyz="-.2 0 -.2" rpy="0 0.785 0"/>
     <axis xyz="0 1 0" />
     <parent link="arm_front"/>
     <child link="stereo_camera_front"/>
-  </joint>
-  <joint name="camera_back_joint" type="fixed">
-    <origin xyz="-.5 0.005 0" rpy="0 -0.785 3.14"/>
-    <axis xyz="0 1 0" />
-    <parent link="arm_back" />
-    <child link="stereo_camera_back"/>
   </joint>
   <joint type="continuous" name="left_wheel_front_hinge">

Commit message: New Sim Package

File: packages/simulation/ez_rassor_description/urdf/ez_rassor.xacro (robot description, xacro)
@@ -1,5 +1,5 @@
 <?xml version='1.0'?>
 <robot name="ez_rassor" xmlns:xacro="http://www.ros.org/wiki/xacro">
-  <xacro:property name="cameraSize" value="0.005"/>
+  <xacro:property name="cameraSize" value="0.05"/>
   <xacro:property name="cameraMass" value="0.1"/>
   <xacro:include filename="$(find ez_rassor_description)/urdf/ez_rassor.gazebo" />
@@ -149,11 +149,11 @@
     </inertial>
   </link>
- <link name="drum_front">
-    <collision name="collision">
+  <link name="drum_front">
+    <!-- <collision name="collision">
       <origin xyz="0 0 0" rpy="0 0 0"/>
       <geometry>
         <robot_arm_drum />
       </geometry>
-    </collision>
+    </collision>-->
     <collision name="collision">
       <origin xyz="0 0 0" rpy="0 1.5707 1.5707"/>
@@ -175,10 +175,10 @@
   </link>
   <link name="drum_back">
-    <collision name="collision">
+    <!-- <collision name="collision">
       <origin xyz="0 0 0" rpy="0 0 3.14159"/>
       <geometry>
         <robot_arm_drum />
       </geometry>
-    </collision>
+    </collision> -->
      <collision name="collision">
       <origin xyz="0 0 0" rpy="0 1.5707 1.5707"/>
@@ -302,5 +302,25 @@
     </inertial>
   </link>
-  <!-- IMU -->
+  <link name="stereo_camera_back">
+    <collision>
+      <origin xyz="0 0 0" rpy="0 0 0"/>
+      <geometry>
+        <box size="${cameraSize} ${cameraSize} ${cameraSize}"/>
+      </geometry>
+    </collision>
+    <visual>
+      <origin xyz="0 0 0" rpy="0 0 0"/>
+      <geometry>
+        <box size="${cameraSize} ${cameraSize} ${cameraSize}"/>
+      </geometry>
+      <material name="green"/>
+    </visual>
+    <inertial>
+      <mass value="${cameraMass}" />
+      <origin xyz="0 0 0" rpy="0 0 0"/>
+      <box_inertia m="${cameraMass}" x="${cameraSize}" y="${cameraSize}" z="${cameraSize}" />
+      <inertia ixx="1e-6" ixy="0" ixz="0" iyy="1e-6" iyz="0" izz="1e-6" />
+    </inertial>
+  </link>
   <link name="imu_link">
     <collision>
@@ -331,8 +351,14 @@
   </joint>
   <joint name="camera_front_joint" type="fixed">
-    <origin xyz="-.2 0 -.2" rpy="0 0.785 0"/>
+    <origin xyz=".5 -0.005 0" rpy="0 0.785 0"/>
     <axis xyz="0 1 0" />
     <parent link="arm_front"/>
     <child link="stereo_camera_front"/>
+  </joint>
+  <joint name="camera_back_joint" type="fixed">
+    <origin xyz="-.5 0.005 0" rpy="0 -0.785 3.14"/>
+    <axis xyz="0 1 0" />
+    <parent link="arm_back" />
+    <child link="stereo_camera_back"/>
   </joint>
   <joint type="continuous" name="left_wheel_front_hinge">

Commit message: Moved camera and fixed the annoying spam bad callback

File: packages/simulation/ez_rassor_description/urdf/ez_rassor.xacro (robot description, xacro)
@@ -1,5 +1,5 @@
 <?xml version='1.0'?>
 <robot name="ez_rassor" xmlns:xacro="http://www.ros.org/wiki/xacro">
-  <xacro:property name="cameraSize" value="0.05"/>
+  <xacro:property name="cameraSize" value="0.04"/>
   <xacro:property name="cameraMass" value="0.1"/>
   <xacro:include filename="$(find ez_rassor_description)/urdf/ez_rassor.gazebo" />
@@ -302,25 +302,4 @@
     </inertial>
   </link>
-  <link name="stereo_camera_back">
-    <collision>
-      <origin xyz="0 0 0" rpy="0 0 0"/>
-      <geometry>
-        <box size="${cameraSize} ${cameraSize} ${cameraSize}"/>
-      </geometry>
-    </collision>
-    <visual>
-      <origin xyz="0 0 0" rpy="0 0 0"/>
-      <geometry>
-        <box size="${cameraSize} ${cameraSize} ${cameraSize}"/>
-      </geometry>
-      <material name="green"/>
-    </visual>
-    <inertial>
-      <mass value="${cameraMass}" />
-      <origin xyz="0 0 0" rpy="0 0 0"/>
-      <box_inertia m="${cameraMass}" x="${cameraSize}" y="${cameraSize}" z="${cameraSize}" />
-      <inertia ixx="1e-6" ixy="0" ixz="0" iyy="1e-6" iyz="0" izz="1e-6" />
-    </inertial>
-  </link>
   <link name="imu_link">
     <collision>
@@ -351,14 +330,8 @@
   </joint>
   <joint name="camera_front_joint" type="fixed">
-    <origin xyz=".5 -0.005 0" rpy="0 0.785 0"/>
+    <origin xyz=".3 0 -.1" rpy="0 0 0"/>
     <axis xyz="0 1 0" />
-    <parent link="arm_front"/>
+    <parent link="base_link"/>
     <child link="stereo_camera_front"/>
-  </joint>
-  <joint name="camera_back_joint" type="fixed">
-    <origin xyz="-.5 0.005 0" rpy="0 -0.785 3.14"/>
-    <axis xyz="0 1 0" />
-    <parent link="arm_back" />
-    <child link="stereo_camera_back"/>
   </joint>
   <joint type="continuous" name="left_wheel_front_hinge">

Commit message: Changed the EZ-RASSOR description slightly to improve traction and physics

File: packages/simulation/ez_rassor_description/urdf/ez_rassor.xacro (robot description, xacro)
@@ -8,4 +8,7 @@
   <!--Below are all of the robot's Links/-->
   <link name='base_link'>
+   <pose>0 0 0 0 0 0</pose>
+  </link>
+  <link name='body'>
     <pose>0 0 0 0 0 0</pose>
     <inertial>
@@ -323,4 +326,10 @@
     </inertial>
   </link>
+  <joint name="body_joint" type="fixed">
+    <axis xyz="0 0 0"/>
+    <origin xyz="0 0 0" rpy="0 0 0"/>
+    <parent link="base_link"/>
+    <child link="body"/>
+  </joint>
   <joint name="imu_joint" type="fixed">
     <axis xyz="0 0 0" />

Commit message: AI is now installable 'maybe'

File: packages/simulation/ez_rassor_description/urdf/ez_rassor.xacro (robot description, xacro)
@@ -13,5 +13,5 @@
     <pose>0 0 0 0 0 0</pose>
     <inertial>
-      <mass value="35.0"/>
+      <mass value="15.0"/>
       <origin xyz="0 0 0" rpy=" 0 0 0"/>
       <inertia
@@ -40,4 +40,16 @@
         <robot_wheel />
       </geometry>
+      <surface>
+        <friction>
+          <mu> .6 </mu>
+          <mu2> .6 </mu2>
+        </friction>
+      </surface>
+      <surface>
+        <friction>
+          <mu> .6 </mu>
+          <mu2> .6 </mu2>
+        </friction>
+      </surface>
     </collision>
     <visual name="left_wheel_front_visual">
@@ -59,4 +71,10 @@
         <robot_wheel />
       </geometry>
+      <surface>
+        <friction>
+        <mu> .6 </mu>
+        <mu2> .6 </mu2>
+        </friction>
+      </surface>
     </collision>
     <visual name="right_wheel_front_visual">
@@ -78,4 +96,10 @@
         <robot_wheel />
       </geometry>
+        <surface>
+          <friction>
+            <mu> .6 </mu>
+            <mu2> .6 </mu2>
+         </friction>
+        </surface>
     </collision>
     <visual name="left_wheel_back_visual">
@@ -97,4 +121,10 @@
         <robot_wheel />
       </geometry>
+      <surface>
+        <friction>
+          <mu> .6 </mu>
+          <mu2> .6 </mu2>
+        </friction>
+      </surface>
     </collision>
     <visual name="right_wheel_back_visual">

Commit message: Hold on to your butts....

File: packages/simulation/ez_rassor_description/urdf/ez_rassor.xacro (robot description, xacro)
@@ -351,7 +351,7 @@
   </joint>
   <joint name="camera_front_joint" type="fixed">
-    <origin xyz=".5 -0.005 0" rpy="0 0.785 0"/>
+    <origin xyz="1 -0.005 0" rpy="0 0 0"/>
     <axis xyz="0 1 0" />
-    <parent link="arm_front"/>
+    <parent link="base_link"/>
     <child link="stereo_camera_front"/>
   </joint>
