Commit message: Renaming EZ-Rassor Description Package and files

File: packages/simulation/ezrassor_sim_description/urdf/ezrassor.xacro (robot description, xacro)
@@ -1,9 +1,9 @@
 <?xml version='1.0'?>
-<robot name="ez_rassor" xmlns:xacro="http://www.ros.org/wiki/xacro">
+<robot name="ezrassor" xmlns:xacro="http://www.ros.org/wiki/xacro">
   <xacro:property name="cameraSize" value="0.05"/>
   <xacro:property name="cameraMass" value="0.1"/>
-  <xacro:include filename="$(find ez_rassor_description)/urdf/ez_rassor.gazebo" />
-  <xacro:include filename="$(find ez_rassor_description)/urdf/materials.xacro" />
-  <xacro:include filename="$(find ez_rassor_description)/urdf/macros.xacro" />
+  <xacro:include filename="$(find ezrassor_sim_description)/urdf/ezrassor.gazebo" />
+  <xacro:include filename="$(find ezrassor_sim_description)/urdf/materials.xacro" />
+  <xacro:include filename="$(find ezrassor_sim_description)/urdf/macros.xacro" />
   <!--Below are all of the robot's Links/-->
   <link name='base_link'>

File: packages/simulation/ezrassor_sim_description/urdf/macros.xacro (robot description, xacro)
@@ -1,4 +1,4 @@
 <?xml version='1.0'?>
-<robot name="ez_rassor" xmlns:xacro="http://www.ros.org/wiki/xacro">
+<robot name="ezrassor" xmlns:xacro="http://www.ros.org/wiki/xacro">
     <!-- Inertia Tensors Used: https://en.wikipedia.org/wiki/List_of_moments_of_inertia#List_of_3D_inertia_tensors -->
     <macro name="cylinder_inertia" params="m r h">
@@ -37,17 +37,17 @@
     <!-- VISUAL AND COLLISION MACROS -->
     <macro name="robot_arm">
-        <mesh filename="package://ez_rassor_description/meshes/drum_arm_short.dae" scale="1.0 1.0 1.0"></mesh>
+        <mesh filename="package://ezrassor_sim_description/meshes/drum_arm_short.dae" scale="1.0 1.0 1.0"></mesh>
     </macro>
     <macro name="robot_arm_drum">
-        <mesh filename="package://ez_rassor_description/meshes/drum.dae" scale="0.35 0.35 0.35"></mesh>
+        <mesh filename="package://ezrassor_sim_description/meshes/drum.dae" scale="0.35 0.35 0.35"></mesh>
     </macro>
     <macro name="robot_wheel">
-        <mesh filename="package://ez_rassor_description/meshes/wheel.dae" scale="0.35 0.35 0.35"></mesh>
+        <mesh filename="package://ezrassor_sim_description/meshes/wheel.dae" scale="0.35 0.35 0.35"></mesh>
     </macro>
     <macro name="base_unit">
-        <mesh filename="package://ez_rassor_description/meshes/base_unit.dae" scale="0.35 0.35 0.35"></mesh>
+        <mesh filename="package://ezrassor_sim_description/meshes/base_unit.dae" scale="0.35 0.35 0.35"></mesh>
     </macro>
     <macro name="drum_arm">
-        <mesh filename="package://ez_rassor_description/meshes/drum_arm.dae" scale="0.35 0.35 0.35"></mesh>
+        <mesh filename="package://ezrassor_sim_description/meshes/drum_arm.dae" scale="0.35 0.35 0.35"></mesh>
     </macro>
 </robot>

File: packages/simulation/ezrassor_sim_description/urdf/materials.xacro (robot description, xacro)
@@ -1,4 +1,4 @@
 <?xml version='1.0'?>
-<robot name="ez_rassor" xmlns:xacro="http://www.ros.org/wiki/xacro">
+<robot name="ezrassor" xmlns:xacro="http://www.ros.org/wiki/xacro">
   <material name="black">
     <color rgba="0.0 0.0 0.0 1.0"/>

Commit message: Fixed some shit I did wrong

File: packages/simulation/ezrassor_sim_description/urdf/ezrassor.xacro (robot description, xacro)
@@ -1,14 +1,17 @@
 <?xml version='1.0'?>
-<robot name="ezrassor" xmlns:xacro="http://www.ros.org/wiki/xacro">
-  <xacro:property name="cameraSize" value="0.05"/>
+<robot name="ez_rassor" xmlns:xacro="http://www.ros.org/wiki/xacro">
+  <xacro:property name="cameraSize" value="0.04"/>
   <xacro:property name="cameraMass" value="0.1"/>
-  <xacro:include filename="$(find ezrassor_sim_description)/urdf/ezrassor.gazebo" />
-  <xacro:include filename="$(find ezrassor_sim_description)/urdf/materials.xacro" />
-  <xacro:include filename="$(find ezrassor_sim_description)/urdf/macros.xacro" />
+  <xacro:include filename="$(find ez_rassor_description)/urdf/ez_rassor.gazebo" />
+  <xacro:include filename="$(find ez_rassor_description)/urdf/materials.xacro" />
+  <xacro:include filename="$(find ez_rassor_description)/urdf/macros.xacro" />
   <!--Below are all of the robot's Links/-->
   <link name='base_link'>
+   <pose>0 0 0 0 0 0</pose>
+  </link>
+  <link name='body'>
     <pose>0 0 0 0 0 0</pose>
     <inertial>
-      <mass value="35.0"/>
+      <mass value="15.0"/>
       <origin xyz="0 0 0" rpy=" 0 0 0"/>
       <inertia
@@ -37,4 +40,16 @@
         <robot_wheel />
       </geometry>
+      <surface>
+        <friction>
+          <mu> .6 </mu>
+          <mu2> .6 </mu2>
+        </friction>
+      </surface>
+      <surface>
+        <friction>
+          <mu> .6 </mu>
+          <mu2> .6 </mu2>
+        </friction>
+      </surface>
     </collision>
     <visual name="left_wheel_front_visual">
@@ -56,4 +71,10 @@
         <robot_wheel />
       </geometry>
+      <surface>
+        <friction>
+        <mu> .6 </mu>
+        <mu2> .6 </mu2>
+        </friction>
+      </surface>
     </collision>
     <visual name="right_wheel_front_visual">
@@ -75,4 +96,10 @@
         <robot_wheel />
       </geometry>
+        <surface>
+          <friction>
+            <mu> .6 </mu>
+            <mu2> .6 </mu2>
+         </friction>
+        </surface>
     </collision>
     <visual name="left_wheel_back_visual">
@@ -94,4 +121,10 @@
         <robot_wheel />
       </geometry>
+      <surface>
+        <friction>
+          <mu> .6 </mu>
+          <mu2> .6 </mu2>
+        </friction>
+      </surface>
     </collision>
     <visual name="right_wheel_back_visual">
@@ -302,5 +335,5 @@
     </inertial>
   </link>
-  <link name="stereo_camera_back">
+  <link name="imu_link">
     <collision>
       <origin xyz="0 0 0" rpy="0 0 0"/>
@@ -323,25 +356,10 @@
     </inertial>
   </link>
-  <link name="imu_link">
-    <collision>
-      <origin xyz="0 0 0" rpy="0 0 0"/>
-      <geometry>
-        <box size="${cameraSize} ${cameraSize} ${cameraSize}"/>
-      </geometry>
-    </collision>
-    <visual>
-      <origin xyz="0 0 0" rpy="0 0 0"/>
-      <geometry>
-        <box size="${cameraSize} ${cameraSize} ${cameraSize}"/>
-      </geometry>
-      <material name="green"/>
-    </visual>
-    <inertial>
-      <mass value="${cameraMass}" />
-      <origin xyz="0 0 0" rpy="0 0 0"/>
-      <box_inertia m="${cameraMass}" x="${cameraSize}" y="${cameraSize}" z="${cameraSize}" />
-      <inertia ixx="1e-6" ixy="0" ixz="0" iyy="1e-6" iyz="0" izz="1e-6" />
-    </inertial>
-  </link>
+  <joint name="body_joint" type="fixed">
+    <axis xyz="0 0 0"/>
+    <origin xyz="0 0 0" rpy="0 0 0"/>
+    <parent link="base_link"/>
+    <child link="body"/>
+  </joint>
   <joint name="imu_joint" type="fixed">
     <axis xyz="0 0 0" />
@@ -351,14 +369,8 @@
   </joint>
   <joint name="camera_front_joint" type="fixed">
-    <origin xyz=".5 -0.005 0" rpy="0 0.785 0"/>
+    <origin xyz=".3 0 -.1" rpy="0 0 0"/>
     <axis xyz="0 1 0" />
-    <parent link="arm_front"/>
+    <parent link="base_link"/>
     <child link="stereo_camera_front"/>
-  </joint>
-  <joint name="camera_back_joint" type="fixed">
-    <origin xyz="-.5 0.005 0" rpy="0 -0.785 3.14"/>
-    <axis xyz="0 1 0" />
-    <parent link="arm_back" />
-    <child link="stereo_camera_back"/>
   </joint>
   <joint type="continuous" name="left_wheel_front_hinge">

Commit message: some fixes and improvements

File: packages/simulation/ezrassor_sim_description/urdf/ezrassor.xacro (robot description, xacro)
@@ -42,28 +42,72 @@
       <surface>
         <friction>
-          <mu> .6 </mu>
-          <mu2> .6 </mu2>
+          <mu> 100 </mu>
+          <mu2> 100 </mu2>
         </friction>
       </surface>
+    </collision>
+    <visual name="left_wheel_front_visual">
+      <origin xyz="0 0 0" rpy="0 0 0"/>
+      <geometry>
+        <robot_wheel />
+      </geometry>
+    </visual>
+    <inertial>
+      <origin xyz="0 0 0" rpy="0 0 0" />
+      <mass value="5"/>
+      <cylinder_inertia m="5" r="0.18" h="0.2"/>
+    </inertial>
+  </link>
+  <link name="right_wheel_front">
+    <collision name="collision">
+      <origin xyz="0 0 0" rpy="0 0 3.14159"/>
+      <geometry>
+        <robot_wheel />
+      </geometry>
       <surface>
         <friction>
-          <mu> .6 </mu>
-          <mu2> .6 </mu2>
+        <mu> 100 </mu>
+        <mu2> 100 </mu2>
         </friction>
       </surface>
     </collision>
-    <visual name="left_wheel_front_visual">
-      <origin xyz="0 0 0" rpy="0 0 0"/>
-      <geometry>
-        <robot_wheel />
-      </geometry>
-    </visual>
-    <inertial>
-      <origin xyz="0 0 0" rpy="0 0 0" />
+    <visual name="right_wheel_front_visual">
+      <origin xyz="0 0 0" rpy="0 0 3.14159"/>
+      <geometry>
+        <robot_wheel />
+      </geometry>
+    </visual>
+    <inertial>
+      <origin xyz="0 0 0" rpy="0 0 3.14159"/>
       <mass value="5"/>
       <cylinder_inertia m="5" r="0.18" h="0.2"/>
     </inertial>
   </link>
-  <link name="right_wheel_front">
+  <link name="left_wheel_back">
+    <collision name="collision">
+      <origin xyz="0 0 0" rpy="0 0 0"/>
+      <geometry>
+        <robot_wheel />
+      </geometry>
+        <surface>
+          <friction>
+            <mu> 100 </mu>
+            <mu2> 100 </mu2>
+         </friction>
+        </surface>
+    </collision>
+    <visual name="left_wheel_back_visual">
+      <origin xyz="0 0 0" rpy="0 0 0"/>
+      <geometry>
+        <robot_wheel />
+      </geometry>
+    </visual>
+    <inertial>
+      <origin xyz="0 0 0" rpy="0 0 0"/>
+      <mass value="5"/>
+      <cylinder_inertia m="5" r="0.18" h="0.2"/>
+    </inertial>
+  </link>
+  <link name="right_wheel_back">
     <collision name="collision">
       <origin xyz="0 0 0" rpy="0 0 3.14159"/>
@@ -73,56 +117,6 @@
       <surface>
         <friction>
-        <mu> .6 </mu>
-        <mu2> .6 </mu2>
-        </friction>
-      </surface>
-    </collision>
-    <visual name="right_wheel_front_visual">
-      <origin xyz="0 0 0" rpy="0 0 3.14159"/>
-      <geometry>
-        <robot_wheel />
-      </geometry>
-    </visual>
-    <inertial>
-      <origin xyz="0 0 0" rpy="0 0 3.14159"/>
-      <mass value="5"/>
-      <cylinder_inertia m="5" r="0.18" h="0.2"/>
-    </inertial>
-  </link>
-  <link name="left_wheel_back">
-    <collision name="collision">
-      <origin xyz="0 0 0" rpy="0 0 0"/>
-      <geometry>
-        <robot_wheel />
-      </geometry>
-        <surface>
-          <friction>
-            <mu> .6 </mu>
-            <mu2> .6 </mu2>
-         </friction>
-        </surface>
-    </collision>
-    <visual name="left_wheel_back_visual">
-      <origin xyz="0 0 0" rpy="0 0 0"/>
-      <geometry>
-        <robot_wheel />
-      </geometry>
-    </visual>
-    <inertial>
-      <origin xyz="0 0 0" rpy="0 0 0"/>
-      <mass value="5"/>
-      <cylinder_inertia m="5" r="0.18" h="0.2"/>
-    </inertial>
-  </link>
-  <link name="right_wheel_back">
-    <collision name="collision">
-      <origin xyz="0 0 0" rpy="0 0 3.14159"/>
-      <geometry>
-        <robot_wheel />
-      </geometry>
-      <surface>
-        <friction>
-          <mu> .6 </mu>
-          <mu2> .6 </mu2>
+          <mu> 100 </mu>
+          <mu2> 100 </mu2>
         </friction>
       </surface>

Commit message: Adding back old launch Files

File: packages/simulation/ezrassor_sim_description/urdf/ezrassor.xacro (robot description, xacro)
@@ -42,34 +42,40 @@
       <surface>
         <friction>
-          <mu> 100 </mu>
-          <mu2> 100 </mu2>
+          <mu> .6 </mu>
+          <mu2> .6 </mu2>
         </friction>
       </surface>
-    </collision>
-    <visual name="left_wheel_front_visual">
-      <origin xyz="0 0 0" rpy="0 0 0"/>
-      <geometry>
-        <robot_wheel />
-      </geometry>
-    </visual>
-    <inertial>
-      <origin xyz="0 0 0" rpy="0 0 0" />
-      <mass value="5"/>
-      <cylinder_inertia m="5" r="0.18" h="0.2"/>
-    </inertial>
-  </link>
-  <link name="right_wheel_front">
-    <collision name="collision">
-      <origin xyz="0 0 0" rpy="0 0 3.14159"/>
-      <geometry>
-        <robot_wheel />
-      </geometry>
       <surface>
         <friction>
-        <mu> 100 </mu>
-        <mu2> 100 </mu2>
+          <mu> .6 </mu>
+          <mu2> .6 </mu2>
         </friction>
       </surface>
     </collision>
+    <visual name="left_wheel_front_visual">
+      <origin xyz="0 0 0" rpy="0 0 0"/>
+      <geometry>
+        <robot_wheel />
+      </geometry>
+    </visual>
+    <inertial>
+      <origin xyz="0 0 0" rpy="0 0 0" />
+      <mass value="5"/>
+      <cylinder_inertia m="5" r="0.18" h="0.2"/>
+    </inertial>
+  </link>
+  <link name="right_wheel_front">
+    <collision name="collision">
+      <origin xyz="0 0 0" rpy="0 0 3.14159"/>
+      <geometry>
+        <robot_wheel />
+      </geometry>
+      <surface>
+        <friction>
+        <mu> .6 </mu>
+        <mu2> .6 </mu2>
+        </friction>
+      </surface>
+    </collision>
     <visual name="right_wheel_front_visual">
       <origin xyz="0 0 0" rpy="0 0 3.14159"/>
@@ -92,6 +98,6 @@
         <surface>
           <friction>
-            <mu> 100 </mu>
-            <mu2> 100 </mu2>
+            <mu> .6 </mu>
+            <mu2> .6 </mu2>
          </friction>
         </surface>
@@ -117,6 +123,6 @@
       <surface>
         <friction>
-          <mu> 100 </mu>
-          <mu2> 100 </mu2>
+          <mu> .6 </mu>
+          <mu2> .6 </mu2>
         </friction>
       </surface>

Commit message: Autonomy Cleanup for Final Delivery

File: packages/simulation/ezrassor_sim_description/urdf/ezrassor.xacro (robot description, xacro)
@@ -1,5 +1,5 @@
 <?xml version='1.0'?>
 <robot name="ezrassor" xmlns:xacro="http://www.ros.org/wiki/xacro">
-  <xacro:property name="cameraSize" value="0.04"/>
+  <xacro:property name="cameraSize" value="0.01"/>
   <xacro:property name="cameraMass" value="0.1"/>
   <xacro:include filename="$(find ezrassor_sim_description)/urdf/ezrassor.gazebo" />

Commit message: Inverting the Back Drum Arm so commands are distributed evenly

File: packages/simulation/ezrassor_sim_description/urdf/ezrassor.xacro (robot description, xacro)
@@ -161,5 +161,5 @@
   <link name="arm_back">
     <collision name="collision">
-      <origin xyz="0 0 0" rpy="0 0 3.1415"/>
+      <origin xyz="0 0 0" rpy="3.1415 0 3.1415"/>
       <geometry>
         <drum_arm />
@@ -167,5 +167,5 @@
     </collision>
     <visual name="visual">
-      <origin xyz="0 0 0" rpy="0 0 3.1415"/>
+      <origin xyz="0 0 0" rpy="3.1415 0 3.1415"/>
       <geometry>
         <drum_arm />
@@ -221,5 +221,5 @@
     </collision>
     <visual name="drum_back">
-      <origin xyz="0 0 0" rpy="0 0 3.14159"/>
+      <origin xyz="0 0 0" rpy="3.1415 0 3.14159"/>
       <geometry>
         <robot_arm_drum />
@@ -407,5 +407,5 @@
   </joint>
   <joint type="continuous" name="arm_front_hinge">
-    <origin xyz="0.20 0 0" rpy="0 0 0"/>
+    <origin xyz="0.20 0 0" rpy="3.1415 0 0"/>
     <child link="arm_front"/>
     <parent link="base_link"/>
@@ -423,5 +423,5 @@
   </joint>
   <joint type="continuous" name="drum_front_hinge">
-    <origin xyz="0.388245 0 0" rpy="0 0 0"/>
+    <origin xyz="0.388245 0 0" rpy="3.1415 0 0"/>
     <child link="drum_front"/>
     <parent link="arm_front"/>
@@ -431,5 +431,5 @@
   </joint>
   <joint type="continuous" name="drum_back_hinge">
-    <origin xyz="-0.388245 0 0" rpy="0 0 0"/>
+    <origin xyz="-0.388245 0 0" rpy="3.1415 0 0"/>
     <child link="drum_back"/>
     <parent link="arm_back"/>

Commit message: replaced stereo camera with depth camera

File: packages/simulation/ezrassor_sim_description/urdf/ezrassor.xacro (robot description, xacro)
@@ -314,5 +314,5 @@
   </transmission>
   <!-- Front Camera Added -->
-  <link name="stereo_camera_front">
+  <link name="depth_camera_front">
     <collision>
       <origin xyz="0 0 0" rpy="0 0 0"/>
@@ -372,5 +372,5 @@
     <axis xyz="0 1 0" />
     <parent link="base_link"/>
-    <child link="stereo_camera_front"/>
+    <child link="depth_camera_front"/>
   </joint>
   <joint type="continuous" name="left_wheel_front_hinge">

Commit message: replace left_camera_optical_frame with depth_camera_optical_frame to get transform of center of depth camera, remove transform_broadcaster node

File: packages/simulation/ezrassor_sim_description/urdf/ezrassor.xacro (robot description, xacro)
@@ -374,4 +374,10 @@
     <child link="depth_camera_front"/>
   </joint>
+  <joint name="depth_camera_optical_joint" type="fixed">
+	  <origin xyz="0 0 0" rpy="${-pi/2} 0 ${-pi/2}"/>
+	  <parent link="depth_camera_front"/>
+	  <child link="depth_camera_optical_frame"/>
+  </joint>
+  <link name="depth_camera_optical_frame"/>
   <joint type="continuous" name="left_wheel_front_hinge">
     <origin xyz="0.20 0.285 0" rpy="0 0 0"/>

Commit message: mounted depth camera to front drum so that camera is higher

File: packages/simulation/ezrassor_sim_description/urdf/ezrassor.xacro (robot description, xacro)
@@ -369,7 +369,7 @@
   </joint>
   <joint name="camera_front_joint" type="fixed">
-    <origin xyz=".3 0 -.1" rpy="0 0 0"/>
+    <origin xyz=".3 0 -.1" rpy="0 ${pi/2} 0"/>
     <axis xyz="0 1 0" />
-    <parent link="base_link"/>
+    <parent link="drum_front"/>
     <child link="depth_camera_front"/>
   </joint>

Commit message: make camera angle parallel with ground (was slightly downward-facing before)

File: packages/simulation/ezrassor_sim_description/urdf/ezrassor.xacro (robot description, xacro)
@@ -369,5 +369,5 @@
   </joint>
   <joint name="camera_front_joint" type="fixed">
-    <origin xyz=".3 0 -.1" rpy="0 ${pi/2} 0"/>
+    <origin xyz="0 0 -.1" rpy="0 ${88*pi/180} 0"/>
     <axis xyz="0 1 0" />
     <parent link="drum_front"/>

Commit message: Lowered camera

File: packages/simulation/ezrassor_sim_description/urdf/ezrassor.xacro (robot description, xacro)
@@ -369,5 +369,5 @@
   </joint>
   <joint name="camera_front_joint" type="fixed">
-    <origin xyz=".3 0 -.1" rpy="0 ${pi/2} 0"/>
+    <origin xyz="0 0 -.1" rpy="0 ${pi/2} 0"/>
     <axis xyz="0 1 0" />
     <parent link="drum_front"/>

Commit message: Reattach camera to base of robot.

File: packages/simulation/ezrassor_sim_description/urdf/ezrassor.xacro (robot description, xacro)
@@ -369,7 +369,7 @@
   </joint>
   <joint name="camera_front_joint" type="fixed">
-    <origin xyz="0 0 -.1" rpy="0 ${pi/2} 0"/>
+    <origin xyz=".3 0 -.1" rpy="0 0 0"/>
     <axis xyz="0 1 0" />
-    <parent link="drum_front"/>
+    <parent link="base_link"/>
     <child link="depth_camera_front"/>
   </joint>
