Commit message: Prepending Xacro XML tags with <xacro: for simulation urdf files. Using xacro python node in launch file

File: packages/simulation/ezrassor_sim_description/urdf/macros.xacro (robot description, xacro)
@@ -2,5 +2,5 @@
 <robot name="ezrassor" xmlns:xacro="http://www.ros.org/wiki/xacro">
     <!-- Inertia Tensors Used: https://en.wikipedia.org/wiki/List_of_moments_of_inertia#List_of_3D_inertia_tensors -->
-    <macro name="cylinder_inertia" params="m r h">
+    <xacro:macro name="cylinder_inertia" params="m r h">
     <inertia
         ixx="${m*((3*r*r)+(h*h))/12}" ixy = "0"                 ixz = "0"
@@ -8,46 +8,46 @@
                                                             izz="${(m*(r*r))/2}"
     />
-    </macro>
-    <macro name="box_inertia" params="m x y z">
+    </xacro:macro>
+    <xacro:macro name="box_inertia" params="m x y z">
     <inertia  ixx="${m*(y*y+z*z)/12}" ixy = "0" ixz = "0"
         iyy="${m*(x*x+z*z)/12}" iyz = "0"
         izz="${m*(x*x+z*z)/12}"
     />
-    </macro>
-    <macro name="sphere_inertia" params="m r">
+    </xacro:macro>
+    <xacro:macro name="sphere_inertia" params="m r">
     <inertia  ixx="${2*m*r*r/5}" ixy = "0" ixz = "0"
         iyy="${2*m*r*r/5}" iyz = "0"
         izz="${2*m*r*r/5}"
     />
-    </macro>
-    <macro name="slender_rod_along_y_inertia" params="m l mass_about">
-        <if value="${mass_about == 'end'}">
+    </xacro:macro>
+    <xacro:macro name="slender_rod_along_y_inertia" params="m l mass_about">
+        <xacro:if value="${mass_about == 'end'}">
             <inertia
                 ixx="${1/3*m*(l*l)}" ixy = "0"
                 ixz = "0" iyy="0"
                 iyz = "0" izz="${1/3*m*(l*l)}" />
-        </if>
-        <unless value="${mass_about == 'center'}">
+        </xacro:if>
+        <xacro:unless value="${mass_about == 'center'}">
             <inertia
                 ixx="${1/12*m*(l*l)}" ixy = "0"
                 ixz = "0" iyy="0"
                 iyz = "0" izz="${1/12*m*(l*l)}" />
-        </unless>
-    </macro>
+        </xacro:unless>
+    </xacro:macro>
     <!-- VISUAL AND COLLISION MACROS -->
-    <macro name="robot_arm">
+    <xacro:macro name="robot_arm">
         <mesh filename="package://ezrassor_sim_description/meshes/drum_arm_short.dae" scale="1.0 1.0 1.0"></mesh>
-    </macro>
-    <macro name="robot_arm_drum">
+    </xacro:macro>
+    <xacro:macro name="robot_arm_drum">
         <mesh filename="package://ezrassor_sim_description/meshes/drum.dae" scale="0.35 0.35 0.35"></mesh>
-    </macro>
-    <macro name="robot_wheel">
+    </xacro:macro>
+    <xacro:macro name="robot_wheel">
         <mesh filename="package://ezrassor_sim_description/meshes/wheel.dae" scale="0.35 0.35 0.35"></mesh>
-    </macro>
-    <macro name="base_unit">
+    </xacro:macro>
+    <xacro:macro name="base_unit">
         <mesh filename="package://ezrassor_sim_description/meshes/base_unit.dae" scale="0.35 0.35 0.35"></mesh>
-    </macro>
-    <macro name="drum_arm">
+    </xacro:macro>
+    <xacro:macro name="drum_arm">
         <mesh filename="package://ezrassor_sim_description/meshes/drum_arm.dae" scale="0.35 0.35 0.35"></mesh>
-    </macro>
+    </xacro:macro>
 </robot>

Commit message: Adding all package changes/additions

File: packages/simulation/ezrassor_sim_description/urdf/macros.xacro (robot description, xacro)
@@ -51,3 +51,34 @@
         <mesh filename="package://ezrassor_sim_description/meshes/drum_arm.dae" scale="0.35 0.35 0.35"></mesh>
     </xacro:macro>
+<!-- ARM VISUAL AND COLLISION MACROS -->
+    <xacro:macro name="link1">
+        <mesh filename="package://ezrassor_sim_description/meshes/link1.dae" scale="0.35 0.35 0.35"></mesh>
+    </xacro:macro>
+    <xacro:macro name="link2">
+        <mesh filename="package://ezrassor_sim_description/meshes/link2.dae" scale="0.35 0.35 0.35"></mesh>
+    </xacro:macro>
+    <xacro:macro name="link3">
+        <mesh filename="package://ezrassor_sim_description/meshes/link3.dae" scale="0.35 0.35 0.35"></mesh>
+    </xacro:macro>
+    <xacro:macro name="link4">
+        <mesh filename="package://ezrassor_sim_description/meshes/link4.dae" scale="0.35 0.35 0.35"></mesh>
+    </xacro:macro>
+    <xacro:macro name="link5">
+        <mesh filename="package://ezrassor_sim_description/meshes/link5.dae" scale="0.35 0.35 0.35"></mesh>
+    </xacro:macro>
+    <xacro:macro name="link6">
+        <mesh filename="package://ezrassor_sim_description/meshes/link6.1.dae" scale="0.35 0.35 0.45"></mesh>
+    </xacro:macro>
+    <xacro:macro name="arm_camera">
+        <mesh filename="package://ezrassor_sim_description/meshes/arm_camera.dae" scale="0.35 0.35 0.35"></mesh>
+    </xacro:macro>
+    <xacro:macro name="grabber1">
+        <mesh filename="package://ezrassor_sim_description/meshes/grabber1.dae" scale="0.35 0.35 0.35"></mesh>
+    </xacro:macro>
+    <xacro:macro name="grabber2">
+        <mesh filename="package://ezrassor_sim_description/meshes/grabber2.dae" scale="0.35 0.35 0.35"></mesh>
+    </xacro:macro>
+    <xacro:macro name="platform">
+        <mesh filename="package://ezrassor_sim_description/meshes/platform.dae" scale="2 2 2"></mesh>
+    </xacro:macro>
 </robot>
